File: Audio-Reg.brd (EAGLE design)
At the start: 20.3 x 25.4 mm, 18 parts, among them IC1 3.3V, Q1 NPN2SC3422-2, Q2 NPN2SC3325, Q3 PNP2SA1313

Commit message: Vカット
Parts:
- added C10, C14, C15, C16, C20, C21, C22, C26, C27, C28, C32, C33, C34, C38, C39, C40, C44, C45, C46, C50, C51, C52, C56, C57, C58, C62, C63, C64, C68, C69, C70, C8, C9: 0.1u, my_rcl:1608
- added C11, C12, C17, C18, C23, C24, C29, C30, C35, C36, C41, C42, C47, C48, C53, C54, C59, C60, C65, C66, C71, C72: 1u, my_rcl:1608
- added C13, C19, C25, C31, C37, C43, C49, C55, C61, C67, C7, R13, R17, R21, R25, R29, R33, R37, R41, R45, R5, R9: DNP, my_rcl:1608
- added D10, D12, D14, D16, D18, D20, D22, D24, D4, D6, D8: BLUE, my_rcl:D1608
- added D11, D13, D15, D17, D19, D21, D23, D3, D5, D7, D9: RED, my_rcl:D1608
- added IC10, IC11, IC12, IC2, IC3, IC4, IC5, IC6, IC7, IC8, IC9: 3.3V, my_ic:SOT23-5
- added JP10, JP11, JP12, JP13, JP14, JP15, JP16, JP17, JP18, JP19, JP20, JP21, JP22, JP23, JP24, JP3, JP4, JP5, JP6, JP7, JP8, JP9: CON, pinhead:1X03
- added Q10, Q13, Q16, Q19, Q22, Q25, Q28, Q31, Q34, Q4, Q7: NPN2SC3422-2, my_ic:TO126-2
- added Q11, Q14, Q17, Q20, Q23, Q26, Q29, Q32, Q35, Q5, Q8: NPN2SC3325, my_ic:SC59
- added Q12, Q15, Q18, Q21, Q24, Q27, Q30, Q33, Q36, Q6, Q9: PNP2SA1313, my_ic:SC59
- added R10, R14, R18, R22, R26, R30, R34, R38, R42, R46, R6: 0, my_rcl:1608
- added R11, R12, R15, R16, R19, R20, R23, R24, R27, R28, R31, R32, R35, R36, R39, R40, R43, R44, R47, R48, R7, R8: 1k, my_rcl:1608
Connections:
- new net GND1: C8.2, C9.2, D4.K, JP3.2, Q6.3, R5.1
- new net GND10: C62.2, C63.2, D22.K, JP21.2, Q33.3, R41.1
- new net GND11: C68.2, C69.2, D24.K, JP23.2, Q36.3, R45.1
- new net GND2: C14.2, C15.2, D6.K, JP5.2, Q9.3, R9.1
- new net GND3: C20.2, C21.2, D8.K, JP7.2, Q12.3, R13.1
- new net GND4: C26.2, C27.2, D10.K, JP9.2, Q15.3, R17.1
- new net GND5: C32.2, C33.2, D12.K, JP11.2, Q18.3, R21.1
- new net GND6: C38.2, C39.2, D14.K, JP13.2, Q21.3, R25.1
- new net GND7: C44.2, C45.2, D16.K, JP15.2, Q24.3, R29.1
- new net GND8: C50.2, C51.2, D18.K, JP17.2, Q27.3, R33.1
- new net GND9: C56.2, C57.2, D20.K, JP19.2, Q30.3, R37.1
- new net IN1: C9.1, JP3.1, Q4.2, R8.2
- new net IN10: C63.1, JP21.1, Q31.2, R44.2
- new net IN11: C69.1, JP23.1, Q34.2, R48.2
- new net IN2: C15.1, JP5.1, Q7.2, R12.2
- new net IN3: C21.1, JP7.1, Q10.2, R16.2
- new net IN4: C27.1, JP9.1, Q13.2, R20.2
- new net IN5: C33.1, JP11.1, Q16.2, R24.2
- new net IN6: C39.1, JP13.1, Q19.2, R28.2
- new net IN7: C45.1, JP15.1, Q22.2, R32.2
- new net IN8: C51.1, JP17.1, Q25.2, R36.2
- new net IN9: C57.1, JP19.1, Q28.2, R40.2
- new net N$100: C67.2, Q35.1, R45.2, R46.1
- new net N$101: D23.K, D24.A
- new net N$102: D23.A, Q35.2
- new net N$103: C70.1, IC12.3
- new net N$104: C70.2, C71.2, C72.2, IC12.2, JP24.2
- new net N$105: C72.1, IC12.1, IC12.5, JP24.1
- new net N$106: C71.1, IC12.4, JP24.3
- new net N$107: Q34.3, Q36.2, R47.2, R48.1
- new net N$108: Q35.3, Q36.1, R47.1
- new net N$11: D3.K, D4.A
- new net N$12: D3.A, Q5.2
- new net N$13: C10.1, IC2.3
- new net N$14: C10.2, C11.2, C12.2, IC2.2, JP4.2
- new net N$15: C12.1, IC2.1, IC2.5, JP4.1
- new net N$16: C11.1, IC2.4, JP4.3
- new net N$17: Q4.3, Q6.2, R7.2, R8.1
- new net N$18: Q5.3, Q6.1, R7.1
- new net N$19: C13.2, Q8.1, R10.1, R9.2
- new net N$20: D5.K, D6.A
- new net N$21: D5.A, Q8.2
- new net N$22: C16.1, IC3.3
- new net N$23: C16.2, C17.2, C18.2, IC3.2, JP6.2
- new net N$24: C18.1, IC3.1, IC3.5, JP6.1
- new net N$25: C17.1, IC3.4, JP6.3
- new net N$26: Q7.3, Q9.2, R11.2, R12.1
- new net N$27: Q8.3, Q9.1, R11.1
- new net N$28: C19.2, Q11.1, R13.2, R14.1
- new net N$29: D7.K, D8.A
- new net N$30: D7.A, Q11.2
- new net N$31: C22.1, IC4.3
- new net N$32: C22.2, C23.2, C24.2, IC4.2, JP8.2
- new net N$33: C24.1, IC4.1, IC4.5, JP8.1
- new net N$34: C23.1, IC4.4, JP8.3
- new net N$35: Q10.3, Q12.2, R15.2, R16.1
- new net N$36: Q11.3, Q12.1, R15.1
- new net N$37: C25.2, Q14.1, R17.2, R18.1
- new net N$38: D10.A, D9.K
- new net N$39: D9.A, Q14.2
- new net N$40: C28.1, IC5.3
- new net N$41: C28.2, C29.2, C30.2, IC5.2, JP10.2
- new net N$42: C30.1, IC5.1, IC5.5, JP10.1
- new net N$43: C29.1, IC5.4, JP10.3
- new net N$44: Q13.3, Q15.2, R19.2, R20.1
- new net N$45: Q14.3, Q15.1, R19.1
- new net N$46: C31.2, Q17.1, R21.2, R22.1
- new net N$47: D11.K, D12.A
- new net N$48: D11.A, Q17.2
- new net N$49: C34.1, IC6.3
- new net N$5: C7.2, Q5.1, R5.2, R6.1
- new net N$50: C34.2, C35.2, C36.2, IC6.2, JP12.2
- new net N$51: C36.1, IC6.1, IC6.5, JP12.1
- new net N$52: C35.1, IC6.4, JP12.3
- new net N$53: Q16.3, Q18.2, R23.2, R24.1
- new net N$54: Q17.3, Q18.1, R23.1
- new net N$55: C37.2, Q20.1, R25.2, R26.1
- new net N$56: D13.K, D14.A
- new net N$57: D13.A, Q20.2
- new net N$58: C40.1, IC7.3
- new net N$59: C40.2, C41.2, C42.2, IC7.2, JP14.2
- new net N$60: C42.1, IC7.1, IC7.5, JP14.1
- new net N$61: C41.1, IC7.4, JP14.3
- new net N$62: Q19.3, Q21.2, R27.2, R28.1
- new net N$63: Q20.3, Q21.1, R27.1
- new net N$64: C43.2, Q23.1, R29.2, R30.1
- new net N$65: D15.K, D16.A
- new net N$66: D15.A, Q23.2
- new net N$67: C46.1, IC8.3
- new net N$68: C46.2, C47.2, C48.2, IC8.2, JP16.2
- new net N$69: C48.1, IC8.1, IC8.5, JP16.1
- new net N$70: C47.1, IC8.4, JP16.3
- new net N$71: Q22.3, Q24.2, R31.2, R32.1
- new net N$72: Q23.3, Q24.1, R31.1
- new net N$73: C49.2, Q26.1, R33.2, R34.1
- new net N$74: D17.K, D18.A
- new net N$75: D17.A, Q26.2
- new net N$76: C52.1, IC9.3
- new net N$77: C52.2, C53.2, C54.2, IC9.2, JP18.2
- new net N$78: C54.1, IC9.1, IC9.5, JP18.1
- new net N$79: C53.1, IC9.4, JP18.3
- new net N$80: Q25.3, Q27.2, R35.2, R36.1
- new net N$81: Q26.3, Q27.1, R35.1
- new net N$82: C55.2, Q29.1, R37.2, R38.1
- new net N$83: D19.K, D20.A
- new net N$84: D19.A, Q29.2
- new net N$85: C58.1, IC10.3
- new net N$86: C58.2, C59.2, C60.2, IC10.2, JP20.2
- new net N$87: C60.1, IC10.1, IC10.5, JP20.1
- new net N$88: C59.1, IC10.4, JP20.3
- new net N$89: Q28.3, Q30.2, R39.2, R40.1
- new net N$90: Q29.3, Q30.1, R39.1
- new net N$91: C61.2, Q32.1, R41.2, R42.1
- new net N$92: D21.K, D22.A
- new net N$93: D21.A, Q32.2
- new net N$94: C64.1, IC11.3
- new net N$95: C64.2, C65.2, C66.2, IC11.2, JP22.2
- new net N$96: C66.1, IC11.1, IC11.5, JP22.1
- new net N$97: C65.1, IC11.4, JP22.3
- new net N$98: Q31.3, Q33.2, R43.2, R44.1
- new net N$99: Q32.3, Q33.1, R43.1
- new net OUT1: C7.1, C8.1, JP3.3, Q4.1, R6.2
- new net OUT10: C61.1, C62.1, JP21.3, Q31.1, R42.2
- new net OUT11: C67.1, C68.1, JP23.3, Q34.1, R46.2
- new net OUT2: C13.1, C14.1, JP5.3, Q7.1, R10.2
- new net OUT3: C19.1, C20.1, JP7.3, Q10.1, R14.2
- new net OUT4: C25.1, C26.1, JP9.3, Q13.1, R18.2
- new net OUT5: C31.1, C32.1, JP11.3, Q16.1, R22.2
- new net OUT6: C37.1, C38.1, JP13.3, Q19.1, R26.2
- new net OUT7: C43.1, C44.1, JP15.3, Q22.1, R30.2
- new net OUT8: C49.1, C50.1, JP17.3, Q25.1, R34.2
- new net OUT9: C55.1, C56.1, JP19.3, Q28.1, R38.2
Routing:
- net OUT8: track 0.00 -> 20.3 mm
- net OUT4: track 0.00 -> 20.3 mm
- net OUT11: track 0.00 -> 20.3 mm
- net OUT9: track 0.00 -> 20.3 mm
- net OUT10: track 0.00 -> 20.3 mm
- net OUT7: track 0.00 -> 20.3 mm
- net OUT5: track 0.00 -> 20.3 mm
- net OUT3: track 0.00 -> 20.3 mm
- net OUT6: track 0.00 -> 20.3 mm
- net OUT1: track 0.00 -> 20.3 mm
- net OUT2: track 0.00 -> 20.3 mm
- net N$82: track 0.00 -> 16.5 mm, vias 0 -> 2
- net N$73: track 0.00 -> 16.5 mm, vias 0 -> 2
- net N$100: track 0.00 -> 16.5 mm, vias 0 -> 2
- net N$91: track 0.00 -> 16.5 mm, vias 0 -> 2
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Other:
- board size 20.3 x 25.4 mm -> 85.7 x 80 mm
- board text added: "C1"
- board text added: "C2"
- board text added: "C3"
- board text added: "C4"
- board text added: "C5"
- board text added: "C6"
- board text added: "D1"
- board text added: "D2"
- board text added: "IC1"
- board text added: "Q1"
- board text added: "Q2"
- board text added: "Q3"
- board text added: "R1"
- board text added: "R2"
- board text added: "R3"
- board text added: "R4"
- board text added: "V-CUT"
