File: Audio-DAC-A.brd (EAGLE design)
At the start: 90 x 90 mm, 125 parts, among them IC1 7833, IC10 NJM2114, IC11 7812, IC12 7812, IC13 78L09, IC2 7805, IC3 7805, IC4 7833, IC5 7812, IC6 AK4493EQ, IC7 7812, IC8 7912, IC9 NJM2114, Q5 NPN2SC3422, Q6 PNP2SA1359, Q7 NPN2SC3422, Q8 PNP2SA1359, Q9 NPN2SC3325, SW1 12V, X1 22.5792MHz, X2 24.576MHz

Commit message: 回路図を修正
Parts:
- C37, C39: value 1n -> 2n
- C42, C43: value 2700p -> 3300p
- C44, C45: value 1n -> 1000p
- D1, D2, D3, D4: value bias -> 1N4148
- R11, R9: value 1k -> 500
- R14, R15, R4, R6: value 1k -> 2k
Changed lines of the file:
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@@
 <?xml version="1.0" encoding="utf-8"?>
 <!DOCTYPE eagle SYSTEM "eagle.dtd">
-<eagle version="9.6.1">
+<eagle version="9.6.2">
 <drawing>
 <settings>
@@
 <setting verticaltext="up"/>
 </settings>
-<grid distance="12.5" unitdist="mil" unit="mil" style="lines" multiple="4" display="yes" altdistance="5" altunitdist="mil" altunit="mil"/>
+<grid distance="25" unitdist="mil" unit="mil" style="lines" multiple="4" display="yes" altdistance="5" altunitdist="mil" altunit="mil"/>
 <layers>
 <layer number="1" name="Top" color="4" fill="1" visible="yes" active="yes"/>
@@
 <attribute name="VALUE" x="19.38" y="80.54" size="0.8128" layer="27" rot="R180"/>
 </element>
-<element name="C37" library="my_rcl" package="1608" value="1n" x="12.7" y="81.28" smashed="yes" rot="R180">
+<element name="C37" library="my_rcl" package="1608" value="2n" x="12.7" y="81.28" smashed="yes" rot="R180">
 <attribute name="NAME" x="8.56" y="81.01" size="0.8128" layer="25"/>
 <attribute name="VALUE" x="14.3" y="83.08" size="0.8128" layer="27" rot="R180"/>
@@
 <attribute name="VALUE" x="16.84" y="62.76" size="0.8128" layer="27" rot="R180"/>
 </element>
-<element name="C39" library="my_rcl" package="1608" value="1n" x="10.16" y="58.42" smashed="yes" rot="R180">
+<element name="C39" library="my_rcl" package="1608" value="2n" x="10.16" y="58.42" smashed="yes" rot="R180">
 <attribute name="NAME" x="6.02" y="58.15" size="0.8128" layer="25"/>
 <attribute name="VALUE" x="11.76" y="60.22" size="0.8128" layer="27" rot="R180"/>
@@
 <attribute name="VALUE" x="33.76" y="70.79" size="0.8128" layer="28" rot="MR90"/>
 </element>
-<element name="C42" library="my_rcl" package="1608" value="2700p" x="38.1" y="77.47" smashed="yes" rot="R90">
+<element name="C42" library="my_rcl" package="1608" value="3300p" x="38.1" y="77.47" smashed="yes" rot="R90">
 <attribute name="NAME" x="39.065" y="80.28" size="0.8128" layer="25" rot="R180"/>
 <attribute name="VALUE" x="39.9" y="75.87" size="0.8128" layer="27" rot="R90"/>
 </element>
-<element name="C43" library="my_rcl" package="1608" value="2700p" x="34.29" y="60.96" smashed="yes" rot="R180">
+<element name="C43" library="my_rcl" package="1608" value="3300p" x="34.29" y="60.96" smashed="yes" rot="R180">
 <attribute name="NAME" x="35.89" y="59.96" size="0.8128" layer="25" rot="R180"/>
 <attribute name="VALUE" x="35.89" y="62.76" size="0.8128" layer="27" rot="R180"/>
 </element>
-<element name="C44" library="my_rcl" package="1608" value="1n" x="41.91" y="81.28" smashed="yes" rot="R180">
+<element name="C44" library="my_rcl" package="1608" value="1000p" x="41.91" y="81.28" smashed="yes" rot="R180">
 <attribute name="NAME" x="42.875" y="83.455" size="0.8128" layer="25" rot="R180"/>
 <attribute name="VALUE" x="43.51" y="83.08" size="0.8128" layer="27" rot="R180"/>
 </element>
-<element name="C45" library="my_rcl" package="1608" value="1n" x="39.37" y="58.42" smashed="yes" rot="R180">
+<element name="C45" library="my_rcl" package="1608" value="1000p" x="39.37" y="58.42" smashed="yes" rot="R180">
 <attribute name="NAME" x="40.6525" y="57.42" size="0.8128" layer="25" rot="R180"/>
 <attribute name="VALUE" x="40.97" y="60.22" size="0.8128" layer="27" rot="R180"/>
@@
 <attribute name="VALUE" x="15.1892" y="61.2648" size="0.8128" layer="27" ratio="10"/>
 </element>
-<element name="R11" library="my_rcl" package="0207/2V" value="1k" x="15.24" y="58.42" smashed="yes" rot="R180">
+<element name="R11" library="my_rcl" package="0207/2V" value="500" x="15.24" y="58.42" smashed="yes" rot="R180">
 <attribute name="NAME" x="15.2908" y="57.404" size="0.8128" layer="25" ratio="10" rot="R180"/>
 <attribute name="VALUE" x="15.2908" y="60.6552" size="0.8128" layer="27" ratio="10" rot="R180"/>
@@
 <attribute name="VALUE" x="34.2392" y="61.2648" size="0.8128" layer="27" ratio="10"/>
 </element>
-<element name="R14" library="my_rcl" package="0207/2V" value="1k" x="41.91" y="78.74" smashed="yes">
+<element name="R14" library="my_rcl" package="0207/2V" value="2k" x="41.91" y="78.74" smashed="yes">
 <attribute name="NAME" x="45.0215" y="78.0542" size="0.8128" layer="25" ratio="10" rot="R90"/>
 <attribute name="VALUE" x="41.8592" y="76.5048" size="0.8128" layer="27" ratio="10"/>
 </element>
-<element name="R15" library="my_rcl" package="0207/2V" value="1k" x="39.37" y="60.96" smashed="yes">
+<element name="R15" library="my_rcl" package="0207/2V" value="2k" x="39.37" y="60.96" smashed="yes">
 <attribute name="NAME" x="42.4815" y="59.9567" size="0.8128" layer="25" ratio="10" rot="R90"/>
 <attribute name="VALUE" x="39.3192" y="58.7248" size="0.8128" layer="27" ratio="10"/>
@@
 <attribute name="VALUE" x="83.3374" y="58.7756" size="0.8128" layer="27" ratio="10" rot="R270"/>
 </element>
-<element name="R4" library="my_rcl" package="0207/2V" value="1k" x="12.7" y="78.74" smashed="yes">
+<element name="R4" library="my_rcl" package="0207/2V" value="2k" x="12.7" y="78.74" smashed="yes">
 <attribute name="NAME" x="8.8392" y="78.486" size="0.8128" layer="25" ratio="10"/>
 <attribute name="VALUE" x="12.6492" y="76.5048" size="0.8128" layer="27" ratio="10"/>
@@
 <attribute name="VALUE" x="12.6492" y="73.9648" size="0.8128" layer="27" ratio="10"/>
 </element>
-<element name="R6" library="my_rcl" package="0207/2V" value="1k" x="10.16" y="60.96" smashed="yes">
+<element name="R6" library="my_rcl" package="0207/2V" value="2k" x="10.16" y="60.96" smashed="yes">
 <attribute name="NAME" x="6.2992" y="60.706" size="0.8128" layer="25" ratio="10"/>
 <attribute name="VALUE" x="10.1092" y="58.7248" size="0.8128" layer="27" ratio="10"/>
@@
 <attribute name="VALUE" x="17.7292" y="73.9648" size="0.8128" layer="27" ratio="10"/>
 </element>
-<element name="R9" library="my_rcl" package="0207/2V" value="1k" x="17.78" y="81.28" smashed="yes" rot="R180">
+<element name="R9" library="my_rcl" package="0207/2V" value="500" x="17.78" y="81.28" smashed="yes" rot="R180">
 <attribute name="NAME" x="21.6408" y="81.534" size="0.8128" layer="25" ratio="10" rot="R180"/>
 <attribute name="VALUE" x="17.8308" y="83.5152" size="0.8128" layer="27" ratio="10" rot="R180"/>
@@
 <attribute name="VALUE" x="60.9092" y="74.5998" size="0.8128" layer="27" ratio="10"/>
 </element>
-<element name="D1" library="my_rcl" package="D0207/2V" value="bias" x="52.07" y="78.74" smashed="yes" rot="R180">
+<element name="D1" library="my_rcl" package="D0207/2V" value="1N4148" x="52.07" y="78.74" smashed="yes" rot="R180">
 <attribute name="NAME" x="55.9308" y="78.994" size="0.8128" layer="25" ratio="10" rot="R180"/>
 <attribute name="VALUE" x="52.1208" y="80.9752" size="0.8128" layer="27" ratio="10" rot="R180"/>
 </element>
-<element name="D2" library="my_rcl" package="D0207/2V" value="bias" x="62.23" y="78.74" smashed="yes">
+<element name="D2" library="my_rcl" package="D0207/2V" value="1N4148" x="62.23" y="78.74" smashed="yes">
 <attribute name="NAME" x="58.3692" y="78.486" size="0.8128" layer="25" ratio="10"/>
 <attribute name="VALUE" x="62.1792" y="76.5048" size="0.8128" layer="27" ratio="10"/>
 </element>
-<element name="D3" library="my_rcl" package="D0207/2V" value="bias" x="48.26" y="63.5" smashed="yes" rot="R180">
+<element name="D3" library="my_rcl" package="D0207/2V" value="1N4148" x="48.26" y="63.5" smashed="yes" rot="R180">
 <attribute name="NAME" x="50.546" y="64.1858" size="0.8128" layer="25" ratio="10" rot="R270"/>
 <attribute name="VALUE" x="48.3108" y="65.7352" size="0.8128" layer="27" ratio="10" rot="R180"/>
 </element>
-<element name="D4" library="my_rcl" package="D0207/2V" value="bias" x="58.42" y="63.5" smashed="yes">
+<element name="D4" library="my_rcl" package="D0207/2V" value="1N4148" x="58.42" y="63.5" smashed="yes">
 <attribute name="NAME" x="56.134" y="63.1317" size="0.8128" layer="25" ratio="10" rot="R90"/>
 <attribute name="VALUE" x="58.3692" y="61.2648" size="0.8128" layer="27" ratio="10"/>
