File: Audio-DAC.brd (EAGLE design)
At the start: 202 parts, among them CON1 USB-5075BR-04-WH, IC1 3.3V 200mA, IC10 -15V, IC11 3.3V, IC12 LPC1114FDH28, IC13 7812, IC14 5V, IC15 5V, IC16 3.3V, IC17 TC7WH74FU, IC18 AK4495EQ, IC19 TC7WU04FU, IC2 AT32UC3A3256, IC20 9V, IC21 -9V, IC22 OP275, IC3 OCT_BUFFER-SO6, IC4 OCT_BUFFER-SO6, IC5 OCT_BUFFER-SO6, IC6 OCT_BUFFER-SO6, IC7 OCT_BUFFER-SO6, IC8 7805, IC9 15V, Q1 NPN2SC3422, Q2 PNP2SA1359, Q3 NPN2SC3422, Q4 PNP2SA1359, Q5 NPN2SC3325, Q6 NPN2SC3325, SW1 EA2, SW2 EA2, X1 12MHz, X2 22.5792MHz, X3 24.576MHz

Commit message: 配置
Parts:
- removed C41: 0.1u, my_rcl:1608
- removed JP1: VOL, pinhead:1X03
- removed JP2: SWD, pinhead:1X05
- added CON2: SWD_CON, my_connector:SWD_CON
- added CON3: VOL_CON, my_connector:VOL_CON
- added TP23: SDA, my_connector:TESTPIN
- added TP24: SCL, my_connector:TESTPIN
- TP10: value TEST_2 -> TEST_11
- TP11: value TEST_4 -> TEST_10
- TP12: value TEST_6 -> TEST_9
- TP9: value TEST_1 -> TEST_12
- moved R25 217.7 mm to (86.4, 10.2)
- moved TP6 208.5 mm to (81.3, 5.08)
- moved TP19 205.5 mm to (95.2, 90.2)
- moved C70 193.7 mm to (90.8, 82.5)
- moved R24 190.6 mm to (68.6, 10.2), turned to 180 degrees
- moved L2 190.4 mm to (80.0, 78.7)
- moved TP5 189.8 mm to (66.0, 5.08)
- moved C29 189.7 mm to (86.4, 20.3)
- moved L1 182.7 mm to (80.0, 90.2)
- moved IC9 172.4 mm to (63.5, 38.1), turned to 180 degrees
- moved TP21 162.9 mm to (90.2, 92.7)
- moved Q4 162.6 mm to (69.8, 71.8), turned to 180 degrees
- moved R57 162.3 mm to (95.2, 84.5)
- moved R56 158.3 mm to (95.2, 86.4), turned to 180 degrees
- moved TP12 157.8 mm to (41.9, 24.1)
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Connections:
- net N$37 renamed VIN+
- net N$38 renamed VIN-
- removed net TEST_1: IC12.1, TP9.1
- removed net TEST_2: IC12.2, TP10.1
- removed net TEST_4: IC12.4, TP11.1
- removed net TEST_6: IC12.6, TP12.1
- new net N$37: IC12.14, TP9.1
- new net N$38: IC12.11, TP10.1
- new net N$53: IC12.10, TP11.1
- new net N$54: IC12.9, TP12.1
- net +12V: now also C26.1, IC8.1
- net +3V3: now also CON3.1, IC19.6; no longer C41.1, JP1.3
- net GND: now also CON2.3, CON3.3; no longer C41.2, IC19.6, JP1.1, JP2.3
- net I2C_SCL: now also TP24.1
- net I2C_SDA: now also TP23.1
- net N$52: now also CON3.2; no longer JP1.2
- net N$94: now also CON2.1; no longer JP2.1
- net N$95: now also CON2.2; no longer JP2.2
- net N$96: now also CON2.4; no longer JP2.4
- net N$97: now also CON2.5; no longer JP2.5
- net V+: no longer C26.1, IC8.1
Routing:
- net USB_VBUS: track 11.4 -> 29.6 mm
- net D_SCK: track 24.0 -> 39.7 mm, vias 2 -> 1
- net D_DATA: track 6.43 -> 21.7 mm
- net D_LRCLK: track 11.5 -> 25.1 mm
- net USB_D-: track 14.2 -> 26.6 mm
- net USB_D+: track 15.0 -> 26.4 mm
- net VBUS: track 5.28 -> 14.2 mm
- net LED_RED: track 8.56 -> 3.09 mm, vias 1 -> 0
- net N$9: track 1.75 -> 7.16 mm, vias 0 -> 1
- net LED_GREEN: track 7.33 -> 2.36 mm, vias 1 -> 0
- net N$7: track 2.32 -> 7.17 mm, vias 0 -> 1
- net N$11: track 7.08 -> 2.47 mm, vias 1 -> 0
- net D_EN_48K: track 30.8 -> 34.5 mm
- net D_MCLK/2: track 30.3 -> 26.7 mm
- net D_!RST: track 11.8 -> 9.06 mm, vias 1 -> 0
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Other:
- board outline added: 99 x 99 mm

Commit message: べた以外できた
Parts:
- added C1, C41: 0.1u, my_rcl:1608
- moved C30 4.94 mm to (25.4, 42.9), turned to 270 degrees
- moved C64 4.80 mm to (7.94, 81.9)
- moved C65 4.80 mm to (9.84, 81.9)
- moved C27 4.80 mm to (42.7, 40.5), turned to 270 degrees
- moved C34 4.72 mm to (22.9, 46.0), turned to 0 degrees
- moved R36 4.18 mm to (6.03, 81.9)
- moved R37 4.18 mm to (11.7, 81.9)
- moved R42 4.02 mm to (36.8, 76.2), turned to 270 degrees
- moved C62 3.24 mm to (21.0, 81.9)
- moved C63 2.62 mm to (19.1, 81.9)
- moved TP10 2.54 mm to (44.5, 26.7)
- moved TP11 2.54 mm to (41.9, 26.7)
- moved C66 2.54 mm to (48.3, 74.9)
- moved C67 2.54 mm to (43.2, 74.9)
- moved R38 2.54 mm to (48.3, 77.5)
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Connections:
- net GND: now also C1.2, C41.1
- net OPA_+: now also C1.1
- net OPA_-: now also C41.2
Routing:
- net GND: track 0.00 -> 210.6 mm, vias 0 -> 31
- net V+: track 0.00 -> 150.7 mm
- net V-: track 0.00 -> 117.4 mm, vias 0 -> 5
- net +3V3: track 0.00 -> 106.5 mm, vias 0 -> 7
- net +12V: track 0.00 -> 87.8 mm, vias 0 -> 1
- net N$34: track 0.00 -> 62.9 mm
- net DAC_AVDD: track 0.00 -> 61.3 mm, vias 0 -> 1
- net N$44: track 0.00 -> 51.4 mm
- net DAC_VREF: track 0.00 -> 47.6 mm
- net OPA_-: track 0.00 -> 44.1 mm
- net I2C_SCL: track 0.00 -> 42.8 mm, vias 0 -> 3
- net I2C_SDA: track 0.00 -> 42.7 mm, vias 0 -> 1
- net N$45: track 0.00 -> 42.7 mm
- net DAC_MCLK: track 0.00 -> 41.1 mm, vias 0 -> 2
- net N$32: track 0.00 -> 40.5 mm
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- added copper zone on layer 15, net GND
- added copper zone on layer 16, net GND
- added copper zone on layer 2, net GND

Commit message: DDCのフォトカプラ追加
Parts:
- added C71: 10u, my_rcl:2012
- added DECO1: ROBOTECH_WHEEL, my_connector:ROBOTECHWHEEL-9MM
- added IC23: OP275, my_ic:DIL08
- added R58, R60: 10k, my_rcl:1608
- added R59: 1.5k, my_rcl:1608
- C15, C2, C42: value 0.1u -> 10u; device my_rcl:1608 -> my_rcl:2012
- C16, C43: value 10u -> 0.1u; device my_rcl:2012 -> my_rcl:1608
- C3: value 10u -> 22u
- C4: value 22u -> 22p; device my_rcl:2012 -> my_rcl:1608
- C45: value 0.1u -> 100u; device my_rcl:1608 -> my_rcl:E2.5-6.5
- C46, C58: value 100u -> 220u; device my_rcl:E2.5-6.5 -> my_rcl:E2,5-8
- C47: value 220u -> 0.22u; device my_rcl:E2,5-8 -> my_rcl:1608
- C49, C55: value 0.22u -> DNP
- C51, C57: value DNP -> 100u; device my_rcl:1608 -> my_rcl:E2.5-6.5
- C52, C54: value 100u -> 0.22u; device my_rcl:E2.5-6.5 -> my_rcl:1608
- C53: value 0.22u -> 100u; device my_rcl:1608 -> my_rcl:E2.5-6.5
- C59: value 220u -> 100u
- C6: value 22p -> 0.1u
- C61: value 100u -> 0.1u; device my_rcl:E2,5-8 -> my_rcl:1608
- C62: value 2000p -> 0.1u
- C66: value 1000p -> 2000p
- C70: value 10u -> 1000p; device my_rcl:2012 -> my_rcl:1608
- C8: value 0.1u -> 10p
- C9: value 10p -> 0.1u
- CON2: value SWD_CON -> VOL_CON; device my_connector:SWD_CON -> my_connector:VOL_CON
- CON3: value VOL_CON -> SWD_CON; device my_connector:VOL_CON -> my_connector:SWD_CON
- IC10: value -15V -> 15V
- IC11: value 3.3V -> -15V; device my_ic:SOT23-5 -> my_ic:REGULATOR_LED
- IC12: value LPC1114FDH28 -> 3.3V; device my_ic:TSSOP28 -> my_ic:SOT23-5
- IC13: value 7812 -> LPC1114FDH28; device my_ic:TO-220 -> my_ic:TSSOP28
- IC14: value 5V -> 7812; device my_ic:REGULATOR_LED -> my_ic:TO-220
- IC16: value 3.3V -> 5V
- IC17: value TC7WH74FU -> 3.3V; device my_ic:SSOP8-P-0.65 -> my_ic:REGULATOR_LED
- IC18: value AK4495EQ -> TC7WH74FU; device my_ic:LQFP44 -> my_ic:SSOP8-P-0.65
- IC19: value TC7WU04FU -> AK4495EQ; device my_ic:SSOP8-P-0.65 -> my_ic:LQFP44
- IC20: value 9V -> TC7WU04FU; device my_ic:REGULATOR_LED -> my_ic:SSOP8-P-0.65
- IC21: value -9V -> 9V
- IC22: value OP275 -> -9V; device my_ic:DIL08 -> my_ic:REGULATOR_LED
- IC8: value 7805 -> OCT_BUFFER-SO6; device my_ic:P-HSIP3_2.30A -> my_ic:SO6
- IC9: value 15V -> 7805; device my_ic:REGULATOR_LED -> my_ic:P-HSIP3_2.30A
- R23: value 1.5k -> 10k
- R24: value 1 -> 10k; device my_rcl:0207/10 -> my_rcl:1608
- R25: value 1 -> 1.5k; device my_rcl:0207/10 -> my_rcl:1608
- R26, R57: value 10k -> 1.5k
- R27, R28: value 10k -> 1; device my_rcl:1608 -> my_rcl:0207/10
- R29, R30, R31: value 100 -> 10k
- R32, R33: value 37 -> 100
- R34: value 1k -> 100; device my_rcl:0207/2V -> my_rcl:1608
- R35, R36: value 1k -> 37; device my_rcl:0207/2V -> my_rcl:1608
- R38, R39, R40: value 2k -> 1k
- R4, R5: value 33 -> 39
- R42, R43, R44: value 1k -> 2k
- R50, R51, R52: value 1 -> 1k
- R54, R56: value 1.5k -> 1; device my_rcl:1608 -> my_rcl:0207/2V
- R55: value 10k -> 1; device my_rcl:1608 -> my_rcl:0207/2V
- moved R25 82.0 mm to (9.53, 38.7), turned to 180 degrees
- moved C1 80.3 mm to (24.1, 5.40), flipped to the top
- moved R28 66.2 mm to (86.4, 10.2)
- moved IC11 61.3 mm to (83.8, 38.1)
- moved C41 58.9 mm to (6.67, 37.1)
- moved R27 50.6 mm to (66.0, 10.2), turned to 180 degrees
- moved R24 47.2 mm to (27.3, 37.1), turned to 0 degrees
- moved C70 46.9 mm to (45.7, 92.7)
- moved IC20 46.7 mm to (3.81, 37.1), flipped to the bottom
- moved R36 41.2 mm to (14.6, 41.6), turned to 180 degrees
- moved R35 41.2 mm to (8.73, 41.6), turned to 0 degrees
- moved R40 39.9 mm to (11.7, 81.9), turned to 90 degrees
- moved C66 39.0 mm to (9.84, 81.9), turned to 270 degrees
- moved R39 37.4 mm to (6.03, 81.9), turned to 90 degrees
- moved IC9 36.3 mm to (27.6, 43.7), flipped to the bottom, turned to 270 degrees
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- renumbered JP3 to JP1, JP4 to JP2
Connections:
- new net EN_+3V3D: IC1.1, IC8.5, R18.2
- new net EN_DDC: IC13.1, R26.1
- new net N$55: IC8.1, R24.2, R26.2
- net +12V: now also C71.1, IC17.3, IC9.1; no longer C70.1, IC13.3, IC8.1
- net +3V3: now also C41.1, CON2.1, IC12.4, IC13.21, IC13.7, IC18.6, IC18.7, IC18.8, IC20.6, IC20.8, R29.2, R31.2; no longer C42.1, CON3.1, IC11.4, IC12.21, IC12.7, IC17.6, IC17.7, IC17.8, IC19.6, IC19.8, R26.2, R28.2
- net +3V3D: now also C11.1, C13.1, C14.2, C16.2, C17.1, C19.1, C3.1, C6.1, C9.2; no longer C11.2, C12.1, C14.1, C15.2, C17.2, C18.1, C20.1, C4.1, C8.1
- net DAC_!EN_48K: now also IC20.7; no longer IC19.7
- net DAC_AVDD: now also C43.1, C47.1, IC17.1, IC19.13, IC19.14, IC19.40; no longer C45.1, C48.1, IC16.1, IC18.13, IC18.14, IC18.40
- net DAC_DATA: now also R33.1; no longer R30.1
- net DAC_DVDD: now also C42.1, C48.1, IC19.43; no longer C43.1, C49.1, IC18.43
- net DAC_EN_48K: now also IC20.1; no longer IC19.1
- net DAC_LN: now also IC19.33, R40.1; no longer IC18.33, R37.1
- net DAC_LP: now also IC19.34, R39.1; no longer IC18.34, R36.1
- net DAC_LRCLK: now also R34.1; no longer R31.1
- net DAC_MCLK: now also IC18.1, IC19.42, R35.2, R36.2; no longer IC17.1, IC18.42, R32.2, R33.2
- net DAC_MCLK/2: now also IC18.5, R25.1; no longer IC17.5, R23.1
- net DAC_PDN: now also IC13.28, IC19.1, R30.2; no longer IC12.28, IC18.1, R27.2
- net DAC_RN: now also IC19.23, R38.1; no longer IC18.23, R35.1
- net DAC_RP: now also IC19.22, R37.1; no longer IC18.22, R34.1
- net DAC_SCK: now also R32.1; no longer R29.1
- net DAC_VCC: now also C51.+, C52.1, C53.+, C54.1, IC15.1, IC19.24, IC19.25, IC19.31, IC19.32; no longer C52.+, C53.1, C54.+, C55.1, IC14.1, IC18.24, IC18.25, IC18.31, IC18.32
- net DAC_VREF: now also C46.+, C50.2, C56.2, C58.+, IC16.1, IC19.17, IC19.18, IC19.38, IC19.39; no longer C47.+, C51.2, C57.2, C59.+, IC15.1, IC18.17, IC18.18, IC18.38, IC18.39
- net DGND: now also C1.2, C11.2, C14.1, C17.2, C18.1, C19.2, C9.1, IC8.4, R22.1; no longer C11.1, C14.2, C17.1, C18.2, C19.1, C9.2
- net D_!RST: now also C12.1; no longer C13.1
- net GND: now also C41.2, C45.-, C47.2, C50.1, C51.-, C52.2, C53.-, C54.2, C56.1, C57.-, C60.+, C61.2, C62.1, C66.2, C68.2, C71.2, IC12.2, IC13.22, IC13.8, IC17.2, IC18.4, IC19.11, IC19.12, IC19.15, IC19.16, IC19.19, IC19.20, IC19.26, IC19.27, IC19.28, IC19.29, IC19.30, IC19.36, IC19.37, IC19.41, IC19.44, IC19.5, IC19.6, IC20.3, IC20.4, IC22.2, IC9.3, R23.1, R24.1, R30.1, R42.1, R44.1, R58.1, R60.1; no longer C1.2, C41.1, C45.2, C47.-, C50.2, C51.1, C52.-, C53.2, C54.-, C56.2, C57.1, C60.-, C61.+, C62.2, C67.2, C69.2, IC12.22, IC12.8, IC13.2, IC17.4, IC18.11, IC18.12, IC18.15, IC18.16, IC18.19, IC18.20, IC18.26, IC18.27, IC18.28, IC18.29, IC18.30, IC18.36, IC18.37, IC18.41, IC18.44, IC18.5, IC18.6, IC19.3, IC19.4, IC20.2, IC9.2, R22.1, R27.1, R39.1, R41.1, R55.1, R57.1
- net HP_SW: now also IC13.17, R59.2; no longer IC12.17, R56.2
- net I2C_SCL: now also IC13.27, IC19.7, R31.1; no longer IC12.27, IC18.7, R28.1
- net I2C_SDA: now also IC13.5, IC19.8, R29.1; no longer IC12.5, IC18.8, R26.1
- net N$14: now also R22.2; no longer R21.2
- net N$15: now also R19.2; no longer R18.2
- net N$16: now also R20.2; no longer R19.2
- net N$17: now also R21.2; no longer R20.2
- net N$18: now also C1.1; no longer C2.1
- net N$19: now also R25.2; no longer R22.2
- net N$20: now also C70.1, IC23.3, R48.2; no longer C69.1, IC22.3, R45.2
- net N$21: now also C67.2, IC23.6, R45.2; no longer C66.2, IC22.6, R42.2
- net N$22: now also C68.1, IC23.5, R46.2; no longer C67.1, IC22.5, R43.2
- net N$23: now also C69.2, IC23.2, R47.2; no longer C68.2, IC22.2, R44.2
- net N$24: now also C67.1, R41.2, R55.1, R56.2; no longer C66.1, R38.2, R52.1, R53.2
- net N$25: now also R55.2; no longer R52.2
- net N$26: now also R51.1; no longer R48.1
- net N$27: now also IC23.7; no longer IC22.7
- net N$28: now also R56.1; no longer R53.1
- net N$29: now also R52.2; no longer R49.2
- net N$3: now also C5.1; no longer C6.1
- net N$30: now also R54.1; no longer R51.1
- net N$31: now also R53.2; no longer R50.2
- net N$32: now also C69.1, R43.2, R53.1, R54.2; no longer C68.1, R40.2, R50.1, R51.2
- net N$35: now also R57.1, R58.2; no longer R54.1, R55.2
- net N$37: now also IC13.14; no longer IC12.14
- net N$38: now also IC13.11; no longer IC12.11
- net N$39: now also R27.1; no longer R24.1
- net N$4: now also C4.1; no longer C5.1
- net N$40: now also R28.1; no longer R25.1
- net N$41: now also IC19.2, R32.2; no longer IC18.2, R29.2
- net N$42: now also IC19.4, R34.2; no longer IC18.4, R31.2
- net N$43: now also IC19.3, R33.2; no longer IC18.3, R30.2
- net N$44: now also C65.1, R39.2, R43.1, R47.1; no longer C64.1, R36.2, R40.1, R44.1
- net N$45: now also C66.1, R40.2, R44.2, R48.1; no longer C65.1, R37.2, R41.2, R45.1
- net N$46: now also C63.1, R37.2, R41.1, R45.1; no longer C62.1, R34.2, R38.1, R42.1
- net N$47: now also C64.1, R38.2, R42.2, R46.1; no longer C63.1, R35.2, R39.2, R43.1
- net N$48: now also R59.1, R60.2; no longer R56.1, R57.2
- net N$5: now also C8.1; no longer C9.1
- net N$50: now also IC12.3; no longer IC11.3
- net N$51: now also IC12.1, IC12.5, IC9.2; no longer IC11.1, IC11.5, IC8.2
- net N$52: now also CON2.2, IC13.13; no longer CON3.2, IC12.13
- net N$53: now also IC13.10; no longer IC12.10
- net N$54: now also IC13.9; no longer IC12.9
- net N$60: now also R49.1; no longer R46.1
- net N$64: now also R50.2; no longer R47.2
- net N$75: now also IC23.1; no longer IC22.1
- net N$8: now also C15.2, C18.2; no longer C16.2, C19.2
- net N$83: now also R35.1; no longer R32.1
- net N$86: now also R36.1; no longer R33.1
- net N$90: now also IC18.2, IC18.3; no longer IC17.2, IC17.3
- net N$94: now also CON3.1, IC13.3; no longer CON2.1, IC12.3
- net N$95: now also CON3.2, IC13.23; no longer CON2.2, IC12.23
- net N$96: now also CON3.4, IC13.12; no longer CON2.4, IC12.12
- net N$97: now also CON3.5, IC13.16; no longer CON2.5, IC12.16
- net OPA_+: now also C59.+, C61.1, IC21.1, IC23.8; no longer C1.1, C60.+, IC20.1, IC22.8
- net OPA_-: now also C60.-, C62.2, IC22.1, IC23.4; no longer C41.2, C61.-, IC21.1, IC22.4
- net SP_SW: now also IC13.18, R57.2; no longer IC12.18, R54.2
- net USB_VBUS: now also C2.1, C20.1, IC8.6; no longer C3.1, IC1.1
- net V+: now also IC10.1, IC14.1, IC21.3, R49.2, R51.2; no longer IC13.1, IC20.3, IC9.1, R46.2, R48.2
- net V-: now also IC11.1, IC22.3, R50.1, R52.1; no longer IC10.1, IC21.3, R47.1, R49.1
- net VCOM_L: now also C45.+, C49.1, IC19.35; no longer C46.+, C50.1, IC18.35
- net VCOM_R: now also C55.1, C57.+, IC19.21; no longer C56.1, C58.+, IC18.21
- net VIN+: now also IC10.3, R27.2; no longer IC9.3, R24.2
- net VIN-: now also IC11.3, R28.2; no longer IC10.3, R25.2
Routing:
- net EN_+3V3D: track 0.00 -> 26.5 mm
- net DGND: track 65.2 -> 70.0 mm, vias 24 -> 27
- net N$55: track 0.00 -> 4.58 mm
- net GND: track 210.6 -> 214.3 mm, vias 31 -> 48
- net USB_VBUS: track 29.6 -> 33.1 mm
- net +3V3D: track 44.7 -> 47.2 mm
- net EN_DDC: track 0.00 -> 1.94 mm
- net USB_D-: track 26.6 -> 24.9 mm
- net USB_D+: track 26.4 -> 24.8 mm
- net N$5: track 6.39 -> 4.82 mm, vias 1 -> 0
- net N$54: track 20.9 -> 22.2 mm
- net N$37: track 18.0 -> 19.3 mm
- net I2C_SCL: track 42.8 -> 43.9 mm
- net +3V3: track 106.5 -> 105.7 mm
- net N$53: track 15.9 -> 16.5 mm
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- added copper zone on layer 1, net V+
- added copper zone on layer 1, net V-
- added copper zone on layer 1, net VIN+
- added copper zone on layer 1, net VIN-
Other:
- board text added: "Audio DAC ver6"

Commit message: ほぼ完成
Parts:
- moved TP20 3.59 mm to (90.2, 95.2)
- moved TP21 0.63 mm to (90.2, 92.1)
Routing:
- net GND: track 214.3 -> 135.4 mm, vias 48 -> 91
- net +12V: track 87.8 -> 90.6 mm
- added copper zone on layer 1, net DAC_VCC
- added copper zone on layer 1, net DAC_VREF
- added copper zone on layer 1, net GND

Commit message: 微修正
Routing:
- net DAC_MCLK: track 41.1 -> 41.7 mm
- net GND: track 135.4 -> 135.9 mm, vias 91 -> 96
Changed lines of the file:
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@@
 <setting verticaltext="up"/>
 </settings>
-<grid distance="12.5" unitdist="mil" unit="mil" style="lines" multiple="4" display="yes" altdistance="5" altunitdist="mil" altunit="mil"/>
+<grid distance="25" unitdist="mil" unit="mil" style="lines" multiple="4" display="yes" altdistance="5" altunitdist="mil" altunit="mil"/>
 <layers>
 <layer number="1" name="Top" color="4" fill="1" visible="yes" active="yes"/>
@@
 <vertex x="61.9125" y="20.0025"/>
 </polygon>
+<wire x1="23.8125" y1="73.025" x2="23.8125" y2="72.39" width="0.1524" layer="21"/>
+<wire x1="24.13" y1="72.7075" x2="23.495" y2="72.7075" width="0.1524" layer="21"/>
+<wire x1="22.5425" y1="75.08875" x2="23.1775" y2="75.08875" width="0.1524" layer="21"/>
+<wire x1="22.86" y1="75.40625" x2="22.86" y2="74.77125" width="0.1524" layer="21"/>
+<wire x1="9.8425" y1="75.08875" x2="10.4775" y2="75.08875" width="0.1524" layer="21"/>
+<wire x1="10.16" y1="75.40625" x2="10.16" y2="74.77125" width="0.1524" layer="21"/>
+<wire x1="9.2075" y1="73.66" x2="9.2075" y2="73.025" width="0.1524" layer="21"/>
+<wire x1="5.3975" y1="63.02375" x2="6.0325" y2="63.02375" width="0.1524" layer="21"/>
+<wire x1="5.715" y1="63.34125" x2="5.715" y2="62.70625" width="0.1524" layer="21"/>
+<wire x1="9.04875" y1="54.61" x2="9.68375" y2="54.61" width="0.1524" layer="21"/>
+<wire x1="9.36625" y1="54.9275" x2="9.36625" y2="54.2925" width="0.1524" layer="21"/>
 </plain>
 <attributes>
@@
 <via x="11.7475" y="50.95875" extent="1-16" drill="0.35"/>
 <wire x1="4.815" y1="50.95875" x2="5.23875" y2="50.535" width="0.508" layer="1"/>
-<via x="5.23875" y="50.165" extent="1-16" drill="0.35"/>
-<wire x1="5.23875" y1="50.535" x2="5.23875" y2="50.165" width="0.508" layer="1"/>
+<via x="5.23875" y="49.68875" extent="1-16" drill="0.35"/>
+<wire x1="5.23875" y1="50.535" x2="5.23875" y2="49.68875" width="0.508" layer="1"/>
 <wire x1="2.98" y1="43.815" x2="2.98" y2="45.04875" width="0.508" layer="1"/>
 <via x="3.175" y="45.24375" extent="1-16" drill="0.35"/>
@@
 <vertex x="46.99" y="49.53"/>
 <vertex x="49.2125" y="51.7525"/>
-<vertex x="51.1175" y="51.7525"/>
-<vertex x="53.34" y="53.975"/>
-<vertex x="53.34" y="60.96"/>
-<vertex x="57.15" y="64.77"/>
-<vertex x="72.39" y="64.77"/>
-<vertex x="73.66" y="63.5"/>
+<vertex x="51.7525" y="51.7525"/>
+<vertex x="53.34" y="53.34"/>
+<vertex x="53.34" y="58.42"/>
+<vertex x="59.055" y="64.135"/>
+<vertex x="71.755" y="64.135"/>
+<vertex x="73.66" y="62.23"/>
 <vertex x="73.66" y="56.1975"/>
 <vertex x="76.2" y="53.6575"/>
@@
 <via x="2.54" y="33.655" extent="1-16" drill="0.35"/>
 <via x="12.7" y="40.005" extent="1-16" drill="0.35"/>
+<via x="1.27" y="54.61" extent="1-16" drill="0.35"/>
+<via x="1.27" y="45.72" extent="1-16" drill="0.35"/>
+<via x="8.89" y="49.53" extent="1-16" drill="0.35"/>
+<via x="4.445" y="58.42" extent="1-16" drill="0.35"/>
+<via x="2.54" y="60.96" extent="1-16" drill="0.35"/>
 <wire x1="88.9" y1="55.88" x2="92.44" y2="82.2325" width="0" layer="19" extent="1-1"/>
 </signal>
@@
 <wire x1="8.52" y1="63.28875" x2="7.62" y2="63.28875" width="0.3048" layer="1"/>
 <wire x1="9.0425" y1="63.81125" x2="8.52" y2="63.28875" width="0.3048" layer="1"/>
-<wire x1="24.13" y1="56.8325" x2="21.9075" y2="54.61" width="1.27" layer="16"/>
-<wire x1="21.9075" y1="54.61" x2="7.77875" y2="54.61" width="1.27" layer="16"/>
 <wire x1="7.62" y1="63.28875" x2="7.25" y2="63.28875" width="0.508" layer="1"/>
 <wire x1="7.25" y1="63.28875" x2="6.50875" y2="62.5475" width="0.508" layer="1"/>
 <via x="6.50875" y="62.5475" extent="1-16" drill="0.35"/>
-<wire x1="6.50875" y1="62.5475" x2="5.87375" y2="61.9125" width="1.27" layer="16"/>
+<wire x1="5.87375" y1="61.9125" x2="6.50875" y2="62.5475" width="1.27" layer="16"/>
 <wire x1="5.87375" y1="61.9125" x2="5.87375" y2="59.69" width="1.27" layer="16"/>
 <wire x1="5.87375" y1="59.69" x2="7.77875" y2="57.785" width="1.27" layer="16"/>
@@
 <wire x1="22.51" y1="61.41125" x2="24.89875" y2="61.41125" width="0.3048" layer="1"/>
 <wire x1="24.89875" y1="61.41125" x2="24.92375" y2="61.43625" width="0.3048" layer="1"/>
+<wire x1="24.13" y1="56.8325" x2="21.9075" y2="54.61" width="1.905" layer="16"/>
+<wire x1="21.9075" y1="54.61" x2="7.77875" y2="54.61" width="1.905" layer="16"/>
 </signal>
 <signal name="DAC_VREF">
@@
 <contactref element="R35" pad="2"/>
 <contactref element="IC18" pad="1"/>
-<wire x1="10.51" y1="62.21125" x2="9.3475" y2="62.21125" width="0.2032" layer="1"/>
-<wire x1="8.5725" y1="60.6425" x2="7.9375" y2="60.0075" width="0.2032" layer="1"/>
-<wire x1="9.3475" y1="62.21125" x2="8.5725" y2="61.43625" width="0.2032" layer="1"/>
-<wire x1="8.5725" y1="61.43625" x2="8.5725" y2="60.6425" width="0.2032" layer="1"/>
-<wire x1="7.9375" y1="60.0075" x2="4.28625" y2="60.0075" width="0.2032" layer="1"/>
-<wire x1="4.28625" y1="60.0075" x2="3.175" y2="58.89625" width="0.2032" layer="1"/>
 <wire x1="13.705" y1="41.5925" x2="11.43" y2="41.5925" width="0.2032" layer="1"/>
 <wire x1="11.43" y1="41.5925" x2="9.63125" y2="41.5925" width="0.2032" layer="1"/>
-<via x="3.175" y="51.59375" extent="1-16" drill="0.35"/>
-<wire x1="3.175" y1="51.59375" x2="7.46125" y2="51.59375" width="0.2032" layer="16"/>
-<wire x1="7.46125" y1="51.59375" x2="10.16" y2="48.895" width="0.2032" layer="16"/>
-<wire x1="10.16" y1="42.8625" x2="11.43" y2="41.5925" width="0.2032" layer="16"/>
+<via x="2.54" y="50.8" extent="1-16" drill="0.35"/>
 <via x="11.43" y="41.5925" extent="1-16" drill="0.35"/>
-<wire x1="3.175" y1="58.89625" x2="3.175" y2="51.59375" width="0.2032" layer="1"/>
-<wire x1="10.16" y1="48.895" x2="10.16" y2="42.8625" width="0.2032" layer="16"/>
-<wire x1="8.55" y1="38.8475" x2="8.55" y2="39.82375" width="0.2032" layer="16"/>
-<wire x1="10.4775" y1="40.64" x2="11.43" y2="41.5925" width="0.2032" layer="16"/>
-<wire x1="8.55" y1="39.82375" x2="9.36625" y2="40.64" width="0.2032" layer="16"/>
-<wire x1="9.36625" y1="40.64" x2="10.4775" y2="40.64" width="0.2032" layer="16"/>
+<wire x1="8.55" y1="38.8475" x2="8.55" y2="39.9825" width="0.2032" layer="16"/>
+<wire x1="8.55" y1="39.9825" x2="9.2075" y2="40.64" width="0.2032" layer="16" curve="-90"/>
+<wire x1="9.2075" y1="40.64" x2="10.4775" y2="40.64" width="0.2032" layer="16"/>
+<wire x1="10.4775" y1="40.64" x2="11.43" y2="41.5925" width="0.2032" layer="16" curve="90"/>
+<wire x1="11.43" y1="41.5925" x2="10.868734375" y2="42.947515625" width="0.2032" layer="16" curve="45"/>
+<wire x1="10.868734375" y1="42.947515625" x2="10.63625" y2="43.18" width="0.2032" layer="16"/>
+<wire x1="10.00125" y1="44.713025" x2="10.63625" y2="43.18" width="0.2032" layer="16" curve="45"/>
+<wire x1="2.54" y1="50.8" x2="8.255" y2="50.8" width="0.2032" layer="16"/>
+<wire x1="8.255" y1="50.8" x2="10.00125" y2="49.05375" width="0.2032" layer="16" curve="-90"/>
+<wire x1="10.00125" y1="49.05375" x2="10.00125" y2="44.713025" width="0.2032" layer="16"/>
+<wire x1="2.54" y1="50.8" x2="2.54" y2="57.94375" width="0.2032" layer="1"/>
+<wire x1="2.54" y1="57.94375" x2="4.7625" y2="60.16625" width="0.2032" layer="1" curve="-90"/>
+<wire x1="4.7625" y1="60.16625" x2="7.3297375" y2="60.16625" width="0.2032" layer="1"/>
+<wire x1="7.3297375" y1="60.16625" x2="8.09625" y2="60.48375" width="0.2032" layer="1" curve="45"/>
+<wire x1="8.09625" y1="60.48375" x2="8.460246875" y2="60.847746875" width="0.2032" layer="1"/>
+<wire x1="8.460246875" y1="60.847746875" x2="8.5725" y2="61.11875" width="0.2032" layer="1" curve="45"/>
+<wire x1="8.5725" y1="61.11875" x2="8.79700625" y2="61.66075625" width="0.2032" layer="1" curve="-45"/>
+<wire x1="8.79700625" y1="61.66075625" x2="9.002253125" y2="61.866003125" width="0.2032" layer="1"/>
+<wire x1="10.51" y1="62.21125" x2="9.835753125" y2="62.21125" width="0.2032" layer="1"/>
+<wire x1="9.835753125" y1="62.21125" x2="9.002253125" y2="61.866003125" width="0.2032" layer="1" curve="45"/>
 </signal>
 <signal name="DAC_!EN_48K">
