File: Audio-DAC.brd (EAGLE design)
At the start: 97 x 99 mm, 209 parts, among them CON1 USB-B, CON2 VOLUEME, CON3 SWD, IC1 3.3V, IC10 +15V, IC11 -15V, IC12 3.3V, IC13 LPC1114, IC14 +10V, IC15 +5V, IC16 +5V, IC17 +3.3V, IC18 TC7WH74FU, IC2 AT32UC3A3256, IC20 TC7WU04FU, IC21 +10V, IC22 -10V, IC23 OP275, IC3 SI8420, IC4 SI8420, IC5 SI8420, IC6 SI8420, IC7 AK4493EQ, IC9 7805, Q1 NPN2SC3422, Q2 PNP2SA1359, Q3 NPN2SC3422, Q4 PNP2SA1359, Q5 NPN, Q6 NPN, SW1 EA2, SW2 EA2, X1 12MHz, X2 24.576MHz, X3 22.5792MHz

Commit message: AK4490
Parts:
- added HT1, HT2: HEATSINK-2, my_connector:HEATSINK2
- added Q10, Q7: NPN2SC3325, my_ic:SC59
- added Q8, Q9: PNP2SA1313, my_ic:SC59
- D3, D4, D5, D6: value 1N4148 -> 10m; device my_rcl:D0207/2V -> my_rcl:SOD123
- IC23: device my_ic:DIL08 -> my_ic:SOP8
- Q1, Q3: value NPN2SC3422 -> NPN-SOT223; device my_ic:TO126 -> my_ic:SOT223
- Q2, Q4: value PNP2SA1359 -> PNP-SOT223; device my_ic:TO126 -> my_ic:SOT223
- R37, R38, R39, R40, R41, R42, R43, R44, R45, R46, R47, R48: device my_rcl:0207/2V -> my_rcl:1608
- R49, R50, R51, R52: value 1k -> 10k; device my_rcl:0207/2V -> my_rcl:1608
- moved D6 157.4 mm to (-21.6, -22.2)
- moved D5 147.6 mm to (-21.6, -18.4), turned to 0 degrees
- moved D4 128.0 mm to (-10.2, -13.3)
- moved D3 119.0 mm to (-10.2, -9.53), turned to 0 degrees
- moved R49 4.89 mm to (54.3, 82.1)
- moved R50 4.89 mm to (64.5, 82.1)
- moved R51 4.89 mm to (77.2, 82.1)
- moved R52 4.89 mm to (87.3, 82.1)
- moved R53 4.89 mm to (50.5, 83.3)
- moved R54 4.89 mm to (60.6, 83.3)
- moved R55 4.89 mm to (73.3, 83.3)
- moved R56 4.89 mm to (83.5, 83.3)
- moved R45 2.29 mm to (36.8, 78.1)
- moved R46 2.01 mm to (38.7, 78.1)
- moved C68 1.90 mm to (41.9, 76.8)
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Connections:
- removed net N$27: D5.2, D6.1, IC23.7
- removed net N$60: D3.1, Q1.3, R49.1
- removed net N$64: D4.2, Q2.3, R50.2
- removed net N$75: D3.2, D4.1, IC23.1
- new net N$16: D4.1, Q2.1, Q7.2, R50.2
- new net N$49: D3.2, Q1.1, Q8.2, R49.1
- new net N$53: IC23.1, Q7.1, Q8.1
- new net N$54: D6.1, Q10.2, Q4.1, R52.2
- net GND: now also HT1.HT1, HT2.HT1
- net N$25: now also Q3.3; no longer Q3.1
- net N$26: now also IC23.7, Q10.1, Q9.1; no longer D5.1, Q3.3, R51.1
- net N$28: now also Q4.3; no longer Q4.1
- net N$29: now also D5.2, Q3.1, Q9.2, R51.1; no longer D6.2, Q4.3, R52.2
- net N$30: now also Q2.3; no longer Q2.1
- net N$31: now also Q1.3; no longer Q1.1
- net V+: now also D3.1, D5.1, Q1.4, Q10.3, Q3.4, Q7.3
- net V-: now also D4.2, D6.2, Q2.4, Q4.4, Q8.3, Q9.3
Routing:
- net V+: track 140.3 -> 60.8 mm
- net V-: track 143.9 -> 76.2 mm
- net GND: track 114.6 -> 57.3 mm, vias 91 -> 62
- net N$27: track 52.0 -> 0.00 mm, vias 1 -> 0
- net DAC_VREF: track 51.3 -> 0.00 mm
- net DAC_AVDD: track 51.4 -> 1.38 mm
- net N$24: track 54.1 -> 4.83 mm, vias 1 -> 0
- net +12V: track 87.4 -> 44.7 mm
- net DAC_VCC: track 37.0 -> 0.00 mm
- net N$32: track 35.9 -> 0.00 mm
- net OPA_-: track 45.3 -> 16.2 mm
- net N$75: track 23.3 -> 0.00 mm
- net N$21: track 21.3 -> 0.00 mm
- net DAC_RN: track 20.4 -> 0.00 mm
- net DAC_PDN: track 28.9 -> 11.0 mm, vias 2 -> 0
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- removed copper zone on layer 1, net DAC_VCC
- removed copper zone on layer 1, net DAC_VREF
- removed copper zone on layer 1, net GND
- removed copper zone on layer 1, net V+
- removed copper zone on layer 16, net V-

Commit message: PCM1795途中
Parts:
- removed C57: 100u, my_rcl:E2.5-6.5
- removed C58: 220u, my_rcl:E2,5-8
- removed C74: 1u, my_rcl:1608
- removed FB2: FB, my_rcl:1608-J
- removed IC16: +5V, my_ic:REGULATOR_LED
- removed R32, R33, R34: 100, my_rcl:1608-J
- added IC19, IC8: (no value), my_ic:SOP8
- added R17: 10k0.1%, my_rcl:1608
- added R18, R19, R20, R21: (no value), my_rcl:1608
- C40, C45, C53: value 100u -> 0.1u; device my_rcl:E2.5-6.5 -> my_rcl:1608
- C42: value 10u -> 0.1u; device my_rcl:2012 -> my_rcl:1608
- C46: value 220u -> 0.1u; device my_rcl:E2,5-8 -> my_rcl:1608
- C47, C48, C54, C55: value 0.1u -> 100u; device my_rcl:1608 -> my_rcl:E2.5-6.5
- C49, C50, C52: value 0.1u -> (none)
- C51: value 100u -> (none); device my_rcl:E2.5-6.5 -> my_rcl:1608
- C56: value 0.1u -> 10u; device my_rcl:1608 -> my_rcl:2012
- IC7: value AK4493EQ -> PCM1795; device my_ic:LQFP48 -> my_ic:TSSOP28
- moved Q10 146.7 mm to (88.9, 84.5)
- moved Q9 135.2 mm to (77.9, 85.2), turned to 90 degrees
- moved Q8 117.4 mm to (68.9, 84.3)
- moved Q7 105.6 mm to (58.7, 82.1)
- moved TP15 94.8 mm to (-47.9, 41.3), turned to 90 degrees
- moved TP18 92.0 mm to (-45.4, 41.3), turned to 90 degrees
- moved Q6 89.4 mm to (-45.4, 38.4), turned to 90 degrees
- moved TP20 89.3 mm to (-42.9, 41.3), turned to 90 degrees
- moved D7 89.1 mm to (-47.9, 34.6), turned to 270 degrees
- moved D8 88.1 mm to (-46.4, 35.6), turned to 180 degrees
- moved Q5 87.3 mm to (-44.8, 36.8), turned to 0 degrees
- moved R58 84.7 mm to (-44.8, 33.7), turned to 0 degrees
- moved R60 84.7 mm to (-44.8, 33.7), turned to 180 degrees
- moved R57 83.1 mm to (-44.8, 31.8), turned to 180 degrees
- moved R59 83.1 mm to (-44.8, 31.8), turned to 0 degrees
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Connections:
- removed net DAC_AVDD: C40.+, C47.1, FB2.1, FB4.1, IC17.1, IC7.14, IC7.15, IC7.16, IC7.44
- removed net DAC_DVDD: C42.1, C48.1, FB2.2, IC7.48
- removed net DAC_VREF: C46.+, C50.2, C56.2, C58.+, IC16.1, IC7.19, IC7.20, IC7.41, IC7.42
- removed net N$14: C43.1, C44.1, FB4.2, X2.4, X3.4
- removed net N$41: IC7.3, R32.2
- removed net N$42: IC7.5, R34.2
- removed net N$43: IC7.4, R33.2
- removed net VCOM_L: C45.+, C49.1, IC7.38
- removed net VCOM_R: C55.1, C57.+, IC7.23
- new net CLK_VDD: C43.1, C44.1, C56.1, FB4.2, X2.4, X3.4
- new net DAC_VDD: C53.1, C54.+, FB4.1, IC17.1, IC7.3, IC7.9
- new net IOUTL+: C49.1, IC7.25, IC8.2, R18.1
- new net IOUTL-: C50.1, C52.1, IC19.6, IC7.26, IC8.6, R19.1, R21.1
- new net IOUTR+: C51.1, IC19.2, IC7.17, R20.1
- new net IOUTR-: IC7.18
- new net N$27: IC7.20, R17.2
- net +12V: no longer IC16.3
- net DAC_DATA: now also IC5.6, IC7.5; no longer IC5.7, R33.1
- net DAC_EN_48K: now also IC4.6
- net DAC_EN_48K_IN: no longer IC4.7
- net DAC_LN: now also C50.2, IC8.7, R19.2; no longer IC7.35
- net DAC_LP: now also C49.2, IC8.1, R18.2; no longer IC7.36
- net DAC_LRCLK: now also IC5.7, IC7.4; no longer IC5.6, R34.1
- net DAC_MCLK: now also IC3.3, IC7.7; no longer IC7.46
- net DAC_MCLK/2: no longer IC3.2
- net DAC_PDN: no longer IC7.2
- net DAC_RN: now also C52.2, IC19.7, R21.2; no longer IC7.26
- net DAC_RP: now also C51.2, IC19.1, R20.2; no longer IC7.25
- net DAC_SCK: now also IC4.7, IC7.6; no longer IC4.6, R32.1
- net DAC_VCC: now also C40.1, C42.1, C45.1, C46.1, C47.+, C48.+, C55.+, IC7.15, IC7.23; no longer C51.+, C52.1, C53.+, C54.1, IC7.27, IC7.33, IC7.34
- net D_DATA: now also IC5.3; no longer IC5.2
- net D_EN_48K: now also IC4.3; no longer IC4.2
- net D_LRCLK: now also IC5.2; no longer IC5.3
- net D_SCK: now also IC4.2; no longer IC4.3
- net GND: now also C40.2, C45.2, C48.-, C53.2, C54.-, C55.-, C56.2, IC19.3, IC19.5, IC3.2, IC7.10, IC7.11, IC7.16, IC7.19, IC7.24, IC7.27, IC7.8, IC8.3, IC8.5, R17.1; no longer C40.-, C45.-, C46.-, C47.2, C48.2, C49.2, C50.1, C51.-, C52.2, C53.-, C54.2, C55.2, C56.1, C57.-, C58.-, C74.2, IC16.2, IC3.3, IC7.12, IC7.13, IC7.17, IC7.18, IC7.21, IC7.22, IC7.29, IC7.30, IC7.31, IC7.32, IC7.39, IC7.40, IC7.45, IC7.47, IC7.6, IC7.7
- net I2C_SCL: now also IC7.12; no longer IC7.8
- net I2C_SDA: now also IC7.13; no longer IC7.9
- net N$37: now also C46.2, C47.-, IC7.21, IC7.22; no longer C74.1, IC7.1
- net OPA_+: now also IC19.8, IC8.8
- net OPA_-: now also IC19.4, IC8.4
Routing:
- net +3V3: track 112.6 -> 0.00 mm, vias 6 -> 0
- net DGND: track 68.8 -> 0.00 mm, vias 110 -> 0
- net GND: track 57.3 -> 1.95 mm, vias 62 -> 27
- net I2C_SCL: track 38.9 -> 0.00 mm, vias 3 -> 0
- net I2C_SDA: track 32.6 -> 0.00 mm, vias 1 -> 0
- net +12V: track 44.7 -> 15.3 mm
- net DAC_SCK: track 23.2 -> 0.00 mm
- net DAC_MCLK: track 21.5 -> 0.00 mm, vias 1 -> 0
- net N$17: track 21.1 -> 0.00 mm, vias 1 -> 0
- net N$19: track 20.0 -> 0.00 mm, vias 1 -> 0
- net N$36: track 17.9 -> 0.00 mm
- net DAC_!EN_48K: track 17.5 -> 0.00 mm, vias 1 -> 0
- net N$18: track 16.9 -> 0.00 mm
- net V+: track 60.8 -> 45.5 mm
- net N$97: track 14.2 -> 0.00 mm, vias 1 -> 0
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Other:
- board text added: "Audio DAC v8"
- board text removed: "Audio DAC v7"

Commit message: だいたい
Parts:
- removed C68: 1000p, my_rcl:1608
- removed IC12: 3.3V, my_ic:SOT23-5
- removed R45, R46, R47, R48: 150, my_rcl:1608
- removed TP24: SCL, my_connector:TESTPIN
- added C57: 0.1u, my_rcl:1608
- added C58: 100u, my_rcl:E2.5-6.5
- added FB2, FB5, FB6: FB, my_rcl:1608-J
- added R22, R23, R24, R25: 10, my_rcl:1608-J
- added R26, R32: 47, my_rcl:1608-J
- added TP21: V-, my_connector:TESTPIN-BIG
- added TP22: GND, my_connector:TESTPIN-BIG
- C26: device my_rcl:1608 -> my_rcl:2012
- C30: value 22u -> 0.1u; device my_rcl:2012 -> my_rcl:1608
- C35, C36: device my_rcl:E5-13 -> my_rcl:E5-10
- C49, C50, C51, C52: value (none) -> 3300p
- C63: value 10n -> 1000p
- C64, C65, C66: value 10n -> 10u; device my_rcl:1608 -> my_rcl:2012
- IC14: value +10V -> +12V
- IC9: value 7805 -> 7803
- Q10, Q7: value NPN2SC3325 -> NPN
- Q8, Q9: value PNP2SA1313 -> PNP
- R18, R19, R20, R21: value (none) -> 1k
- R30: value 10k -> 47; device my_rcl:1608 -> my_rcl:1608-J
- R37, R38, R39, R40: value 2k -> 1k
- R41, R42, R43, R44: value 4k -> 1k
- TP11: value SDA -> V+; device my_connector:TESTPIN -> my_connector:TESTPIN-BIG
- moved D4 132.8 mm to (81.4, 82.9), turned to 270 degrees
- moved D6 132.5 mm to (59.5, 82.5), turned to 270 degrees
- moved D5 123.3 mm to (48.9, 82.7), turned to 90 degrees
- moved D3 122.4 mm to (70.0, 83.0), turned to 90 degrees
- moved R17 116.3 mm to (17.9, 62.4), turned to 90 degrees
- moved TP15 96.9 mm to (48.9, 45.7), turned to 0 degrees
- moved FB3 94.6 mm to (45.7, 46.8), flipped to the top, turned to 0 degrees
- moved TP18 94.3 mm to (48.9, 40.6), turned to 0 degrees
- moved C26 93.8 mm to (45.7, 44.8), flipped to the top, turned to 180 degrees
- moved R59 92.0 mm to (47.1, 35.4), flipped to the bottom, turned to 90 degrees
- moved TP20 91.8 mm to (48.9, 43.2), turned to 0 degrees
- moved D8 91.0 mm to (44.6, 38.3), flipped to the bottom, turned to 0 degrees
- moved Q6 89.8 mm to (44.3, 34.6), flipped to the bottom, turned to 0 degrees
- moved R60 89.1 mm to (44.3, 31.4), flipped to the bottom
- moved CON2 88.4 mm to (49.4, 35.1), turned to 270 degrees
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Connections:
- net N$24 renamed AMP_ROUT
- net N$32 renamed AMP_LOUT
- net N$94 renamed SWCLK
- net N$95 renamed LPC_NRST
- net N$96 renamed SWDIO
- net N$97 renamed LPC_UART_TX
- removed net DAC_PDN: IC13.28, R30.2
- removed net N$46: C63.1, R37.2, R41.1, R45.1
- removed net N$50: C34.1, IC12.3
- removed net N$51: C30.1, IC12.1, IC12.5, IC9.3
- removed net N$56: C26.1, FB3.2, IC9.1
- new net +12VD: C26.1, D7.2, D8.2, FB3.2, IC9.1, SW1.10, SW2.10, TP15.1, TP16.1
- new net DAC_LRCLK_IN: IC5.7, R15.1, R30.1
- new net N$14: C58.-, IC7.21
- new net N$24: C66.1, FB6.2, IC14.3
- new net N$32: IC5.6, R32.1
- new net N$41: C49.1, IC8.2, R18.1, R22.2
- new net N$42: C50.1, IC8.6, R19.1, R23.2
- new net N$43: C51.1, IC19.2, R20.1, R24.2
- new net N$55: C52.1, IC19.6, R21.1, R25.2
- net +12V: no longer D7.2, D8.2, SW1.10, SW2.10, TP15.1, TP16.1
- net +3V3: now also IC9.3; no longer IC12.4
- net DAC_DATA: now also R32.2; no longer IC5.6
- net DAC_EN_48K: no longer IC4.6
- net DAC_EN_48K_IN: now also IC4.6
- net DAC_LN: now also C52.2, IC19.7, R21.2; no longer C50.2, IC8.7, R19.2
- net DAC_LP: now also C51.2, IC19.1, R20.2; no longer C49.2, IC8.1, R18.2
- net DAC_LRCLK: now also R30.2; no longer IC5.7, R15.1
- net DAC_MCLK: no longer IC3.3
- net DAC_MCLK/2: now also IC3.3
- net DAC_RN: now also C50.2, IC8.7, R19.2; no longer C52.2, IC19.7, R21.2
- net DAC_RP: now also C49.2, IC8.1, R18.2; no longer C51.2, IC19.1, R20.2
- net DAC_SCK: now also R26.2; no longer IC4.7
- net DAC_VCC: now also C58.+; no longer C46.1
- net GND: now also C46.1, C57.1, C65.1, TP22.1; no longer C65.2, C68.2, IC12.2, R30.1
- net I2C_SCL: no longer TP24.1
- net I2C_SDA: no longer TP11.1
- net IOUTL+: now also R25.1; no longer C49.1, IC8.2, R18.1
- net IOUTL-: now also R24.1; no longer C50.1, C52.1, IC19.6, IC8.6, R19.1, R21.1
- net IOUTR+: now also R23.1; no longer C51.1, IC19.2, R20.1
- net IOUTR-: now also R22.1
- net N$20: now also C64.1, FB2.2, IC21.3; no longer C70.1, IC23.3, R48.2
- net N$21: now also R37.2, R41.1; no longer R45.2
- net N$22: now also C63.1, R38.2, R42.2; no longer C68.1, R46.2
- net N$23: now also C65.2, FB5.2, IC22.3; no longer C69.2, IC23.2, R47.2
- net N$33: now also SW1.7; no longer SW1.4
- net N$34: now also SW1.4; no longer SW1.7
- net N$37: no longer C46.2, IC7.21
- net N$44: now also C69.2, IC23.2; no longer C65.1, R47.1
- net N$45: now also C70.1, IC23.3; no longer C66.1, R48.1
- net N$47: now also IC4.7, R26.1; no longer C64.1, R38.2, R42.2, R46.1
- net OPA_+: now also C30.1, C34.1
- net OPA_-: now also C46.2, C57.2
- net SPK_L: now also SW1.3; no longer SW1.8
- net SPK_R: now also SW1.8; no longer SW1.3
- net V+: now also FB2.1, FB6.1, TP11.1; no longer IC14.3, IC21.3
- net V-: now also FB5.1, TP21.1; no longer IC22.3
Routing:
- net +3V3: track 0.00 -> 90.0 mm, vias 0 -> 5
- net OPA_-: track 16.2 -> 88.4 mm, vias 0 -> 3
- net DAC_VCC: track 0.00 -> 68.9 mm
- net AMP_LOUT: track 0.00 -> 61.2 mm, vias 0 -> 1
- net N$53: track 0.00 -> 48.4 mm, vias 0 -> 2
- net OPA_+: track 22.0 -> 69.8 mm, vias 0 -> 3
- net V+: track 45.5 -> 88.2 mm, vias 0 -> 91
- net V-: track 64.2 -> 106.8 mm, vias 0 -> 100
- net AMP_ROUT: track 4.83 -> 47.2 mm, vias 0 -> 1
- net N$38: track 0.00 -> 38.6 mm, vias 0 -> 2
- net I2C_SDA: track 0.00 -> 38.5 mm, vias 0 -> 2
- net DAC_LP: track 0.05 -> 36.7 mm
- net I2C_SCL: track 0.00 -> 35.1 mm, vias 0 -> 2
- net DAC_LN: track 0.00 -> 33.7 mm
- net CLK_VDD: track 0.00 -> 33.0 mm
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- added copper zone on layer 16, net DAC_VCC
- added copper zone on layer 1, net GND
- added copper zone on layer 1, net V+
- added copper zone on layer 16, net V+
- added copper zone on layer 2, net V+
- added copper zone on layer 1, net V-
- added copper zone on layer 15, net V-
- added copper zone on layer 16, net V-
- removed copper zone on layer 15, net GND
- removed copper zone on layer 16, net GND
- removed copper zone on layer 2, net GND
- removed copper zone on layer 1, net VIN+
- removed copper zone on layer 1, net VIN-
