File: Audio-DAC.brd (EAGLE design)
At the start: 97 x 99 mm, 220 parts, among them CON1 USB-B, CON2 VOLUEME, CON3 SWD, IC1 3.3V, IC10 +15V, IC11 -15V, IC13 LPC1114, IC14 +12V, IC15 +5V, IC17 +3.3V, IC18 TC7WH74FU, IC2 AT32UC3A3256, IC20 TC7WU04FU, IC21 +10V, IC22 -10V, IC23 OP275, IC3 SI8420, IC4 SI8420, IC5 SI8420, IC6 SI8420, IC7 PCM1795, IC9 7803, Q1 NPN-SOT223, Q10 NPN, Q2 PNP-SOT223, Q3 NPN-SOT223, Q4 PNP-SOT223, Q5 NPN, Q6 NPN, Q7 NPN, Q8 PNP, Q9 PNP, SW1 EA2, SW2 EA2, X1 12MHz, X2 24.576MHz, X3 22.5792MHz

Commit message: 全部つないだ
Parts:
- IC23: value OP275 -> (none)
- moved TP13 5.08 mm to (46.4, 22.9)
- moved TP12 3.71 mm to (46.4, 25.6)
- moved TP23 2.54 mm to (48.9, 22.9)
- moved TP14 2.54 mm to (48.9, 25.4)
- moved R15 0.79 mm to (3.17, 35.6)
- moved IC20 0.16 mm to (14.6, 37.1)
Routing:
- net GND: track 0.00 -> 84.6 mm, vias 0 -> 46
- net DGND: track 0.00 -> 26.3 mm, vias 0 -> 1
- net +12V: track 30.5 -> 36.1 mm
- net N$17: track 12.0 -> 8.70 mm
- net N$18: track 13.6 -> 11.1 mm
- net N$19: track 10.5 -> 8.01 mm
- net N$38: track 38.6 -> 41.0 mm
- net DAC_LP: track 36.7 -> 35.1 mm
- net +3V3: track 90.0 -> 91.2 mm
- net DAC_MCLK/2: track 5.13 -> 6.08 mm
- net DAC_LRCLK_IN: track 6.85 -> 6.06 mm
- net OPA_-: track 88.4 -> 89.0 mm
- net DAC_EN_48K: track 6.55 -> 7.07 mm
- added copper zone on layer 16, net GND
- added copper zone on layer 2, net GND

Commit message: バージョン
Routing:
- net DAC_LN: track 34.1 -> 33.2 mm
Changed lines of the file:
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@@
 <wire x1="97" y1="99" x2="0" y2="99" width="0.2032" layer="20" locked="yes"/>
 <wire x1="0" y1="99" x2="0" y2="0" width="0.2032" layer="20" locked="yes"/>
-<text x="40.64" y="17.145" size="2.54" layer="1" font="vector" ratio="12">Audio DAC v8</text>
+<text x="40.3225" y="16.03375" size="2.54" layer="1" font="vector" ratio="12">Audio DAC v8</text>
 <polygon width="0.2032" layer="29">
-<vertex x="40.3225" y="20.0025"/>
-<vertex x="40.3225" y="16.8275"/>
-<vertex x="61.11875" y="16.8275"/>
-<vertex x="61.11875" y="20.0025"/>
+<vertex x="40.005" y="18.89125"/>
+<vertex x="40.005" y="15.71625"/>
+<vertex x="60.80125" y="15.71625"/>
+<vertex x="60.80125" y="18.89125"/>
 </polygon>
 <wire x1="8.73125" y1="23.495" x2="8.73125" y2="22.5425" width="0.0508" layer="42"/>
@@
 <wire x1="5.715" y1="26.3525" x2="5.715" y2="25.7175" width="0.127" layer="21"/>
 <wire x1="17.93875" y1="53.18125" x2="17.93875" y2="52.705" width="0.1524" layer="41"/>
+<wire x1="40.005" y1="18.89125" x2="40.005" y2="15.71625" width="0.2032" layer="41"/>
+<wire x1="40.005" y1="15.71625" x2="60.80125" y2="15.71625" width="0.2032" layer="41"/>
+<wire x1="60.80125" y1="15.71625" x2="60.80125" y2="18.89125" width="0.2032" layer="41"/>
+<wire x1="60.80125" y1="18.89125" x2="40.005" y2="18.89125" width="0.2032" layer="41"/>
 </plain>
 <attributes>
@@
 <wire x1="3.96875" y1="77.89375" x2="4.18" y2="78.105" width="0.3048" layer="1"/>
 <wire x1="4.18" y1="78.105" x2="6.29" y2="78.105" width="0.3048" layer="1"/>
-<wire x1="6.29" y1="78.105" x2="6.29" y2="79.95" width="0.3048" layer="1"/>
-<wire x1="6.29" y1="79.95" x2="14.605" y2="88.265" width="0.3048" layer="1"/>
+<wire x1="6.29" y1="78.105" x2="6.29" y2="79.6325" width="0.3048" layer="1"/>
+<wire x1="6.29" y1="79.6325" x2="14.9225" y2="88.265" width="0.3048" layer="1"/>
 <wire x1="30.5325" y1="88.265" x2="31.32625" y2="89.05875" width="0.3048" layer="1"/>
-<wire x1="14.605" y1="88.265" x2="30.5325" y2="88.265" width="0.3048" layer="1"/>
+<wire x1="14.9225" y1="88.265" x2="30.5325" y2="88.265" width="0.3048" layer="1"/>
 </signal>
 <signal name="DAC_LN">
@@
 <wire x1="11.49" y1="76.835" x2="12.065" y2="76.835" width="0.3048" layer="1"/>
 <wire x1="12.065" y1="76.835" x2="12.85875" y2="77.62875" width="0.3048" layer="1"/>
-<wire x1="12.85875" y1="77.62875" x2="12.85875" y2="85.725" width="0.3048" layer="1"/>
-<wire x1="12.85875" y1="85.725" x2="14.76375" y2="87.63" width="0.3048" layer="1"/>
-<wire x1="30.85" y1="87.63" x2="31.485" y2="86.995" width="0.3048" layer="1"/>
-<wire x1="14.76375" y1="87.63" x2="30.85" y2="87.63" width="0.3048" layer="1"/>
+<wire x1="12.85875" y1="77.62875" x2="12.85875" y2="84.7725" width="0.3048" layer="1"/>
+<wire x1="12.85875" y1="84.7725" x2="15.24" y2="87.15375" width="0.3048" layer="1"/>
+<wire x1="31.32625" y1="87.15375" x2="31.485" y2="86.995" width="0.3048" layer="1"/>
+<wire x1="15.24" y1="87.15375" x2="31.32625" y2="87.15375" width="0.3048" layer="1"/>
 </signal>
 <signal name="DAC_RN">

Commit message: シルク整えた
Parts:
- added C68, C71: FF, my_rcl:1608
- TP12: value TEST_9 -> TP9
- TP13: value TEST_10 -> TP10
- TP14: value TEST_14 -> TP14
- TP23: value TEST_11 -> TP11
- moved R50 2.23 mm to (77.0, 82.9)
- moved R54 2.23 mm to (84.9, 82.9)
- moved D4 2.23 mm to (79.2, 83.0)
- moved Q8 2.23 mm to (82.1, 83.0)
- moved D5 2.06 mm to (46.8, 82.7)
- moved D6 2.06 mm to (57.5, 82.5)
- moved Q10 2.06 mm to (49.7, 82.7)
- moved Q9 2.06 mm to (60.2, 82.4)
- moved R51 2.06 mm to (44.8, 83.0)
- moved R52 2.06 mm to (55.4, 82.5)
- moved R55 2.06 mm to (52.5, 82.7)
- moved R56 2.06 mm to (63.3, 82.7)
- moved D3 1.75 mm to (68.3, 83.0)
- moved Q7 1.75 mm to (71.1, 82.9)
- moved R49 1.75 mm to (66.2, 83.0)
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Connections:
- net AMP_LOUT: now also C68.1
- net AMP_ROUT: now also C71.1
- net N$26: now also C71.2
- net N$53: now also C68.2
Routing:
- net AMP_ROUT: track 47.2 -> 49.7 mm
- net N$53: track 48.4 -> 47.3 mm
- net N$30: track 4.00 -> 2.92 mm
- net AMP_LOUT: track 61.2 -> 62.2 mm
- net N$25: track 3.77 -> 2.92 mm
- net N$28: track 3.93 -> 3.07 mm
- net DAC_LN: track 33.2 -> 32.4 mm
- net DAC_LP: track 34.9 -> 34.1 mm
- net V+: track 88.2 -> 87.4 mm, vias 91 -> 88
- net N$31: track 3.80 -> 3.07 mm
- net N$16: track 12.0 -> 11.4 mm
- net V-: track 106.8 -> 106.3 mm, vias 100 -> 90
- added copper zone on layer 2, net N$46
- added copper zone on layer 2, net N$50
- added copper zone on layer 15, net V+

Commit message: 微修正
Parts:
- removed TP15, TP16: +12V, my_connector:TESTPIN
- removed TP17, TP20: SW_SP, my_connector:TESTPIN
- removed TP18, TP19: SW_HP, my_connector:TESTPIN
- TP31: value GND_L -> GND
- moved C72 0.95 mm to (7.46, 36.7)
- moved C59 0.64 mm to (38.7, 69.2)
- moved C60 0.64 mm to (47.6, 69.2)
- moved C61 0.64 mm to (41.9, 81.9)
- moved C62 0.64 mm to (34.0, 84.0)
- moved C68 0.64 mm to (41.9, 86.0)
- moved C63 0.63 mm to (36.7, 77.8)
- moved C67 0.63 mm to (40.5, 75.7)
- moved C69 0.63 mm to (39.2, 87.6)
- moved C70 0.63 mm to (35.2, 87.6)
- moved C71 0.63 mm to (43.3, 76.8)
- moved IC23 0.63 mm to (37.9, 82.7)
- moved R37 0.63 mm to (32.9, 77.8)
- moved R38 0.63 mm to (32.9, 75.7)
- moved R39 0.63 mm to (31.4, 89.7)
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Connections:
- net +12VD: no longer TP15.1, TP16.1
- net HP_L: now also SW2.8; no longer SW2.3
- net HP_R: now also SW2.3; no longer SW2.8
- net N$33: now also SW1.4, SW2.4; no longer SW1.7, SW2.7
- net N$34: now also SW1.7, SW2.7; no longer SW1.4, SW2.4
- net SPK_L: now also SW1.8; no longer SW1.3
- net SPK_R: now also SW1.3; no longer SW1.8
- net SW_HP: no longer TP18.1, TP19.1
- net SW_SP: no longer TP17.1, TP20.1
Routing:
- net SW_HP: track 10.6 -> 53.8 mm, vias 0 -> 1
- net +12VD: track 32.8 -> 70.1 mm, vias 0 -> 2
- net SW_SP: track 20.6 -> 51.3 mm, vias 0 -> 1
- net N$34: track 48.0 -> 37.7 mm
- net N$33: track 44.3 -> 34.1 mm
- net GND: track 84.6 -> 91.1 mm, vias 46 -> 121
- net AMP_ROUT: track 49.7 -> 47.7 mm
- net V-: track 106.3 -> 107.5 mm
- net OPA_+: track 69.8 -> 70.8 mm
- net +3V3: track 91.2 -> 91.9 mm
- net AMP_LOUT: track 62.2 -> 62.9 mm
- net V+: track 87.4 -> 86.7 mm
- net N$26: track 26.5 -> 25.9 mm
- net DAC_LN: track 32.4 -> 32.9 mm
- net OPA_-: track 89.0 -> 88.5 mm
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- added copper zone on layer 15, net GND
- added copper zone on layer 15, net N$46
- added copper zone on layer 15, net N$50
- added copper zone on layer 2, net V-
- added copper zone on layer 16, net VIN+
- added copper zone on layer 16, net VIN-
- removed copper zone on layer 2, net N$46
- removed copper zone on layer 2, net N$50
- removed copper zone on layer 15, net V-

Commit message: Add 位相補償
Parts:
- added C74, C75: CMP, my_rcl:1608
- moved C71 2.06 mm to (45.4, 76.8)
- moved R43 0.35 mm to (38.9, 89.9)
- moved C68 0.32 mm to (41.9, 85.7)
- moved C69 0.32 mm to (38.9, 87.6)
- moved R40 0.32 mm to (31.3, 87.6)
- moved R39 0.22 mm to (31.3, 89.9)
- moved R44 0.22 mm to (35.1, 89.9)
- moved C67 0.16 mm to (40.5, 75.6)
- moved C70 0.16 mm to (35.1, 87.6)
- moved R38 0.16 mm to (32.9, 75.6)
- moved R42 0.16 mm to (36.7, 75.6)
Connections:
- net N$21: now also C75.1
- net N$26: now also C75.2
- net N$44: now also C74.1
- net N$53: now also C74.2
Routing:
- net N$21: track 16.0 -> 21.2 mm
- net N$44: track 11.3 -> 15.9 mm
- net N$53: track 47.2 -> 51.8 mm
- net AMP_ROUT: track 47.7 -> 49.6 mm
- net OPA_-: track 88.5 -> 90.0 mm

Commit message: 微修正
Parts:
- removed DECO1: ROBOTECH_WHEEL, my_connector:ROBOTECHWHEEL-9MM
- added R33, R34, R45, R46: 10, my_rcl:1608
- IC19, IC23, IC8: value (none) -> ADA4075
- R17: value 10k0.1% -> 10k
- moved C54 1.72 mm to (26.7, 50.5)
- moved C56 0.95 mm to (25.9, 42.2), turned to 0 degrees
- moved FB4 0.95 mm to (24.9, 45.1)
- moved Q9 0.35 mm to (60.3, 82.7)
- moved D6 0.32 mm to (57.5, 82.9)
- moved Q8 0.32 mm to (82.1, 82.7)
- moved R51 0.32 mm to (44.8, 82.7)
- moved D5 0.16 mm to (46.8, 82.9)
- moved Q7 0.16 mm to (71.1, 82.7)
- moved R50 0.16 mm to (77.0, 82.7)
- moved R54 0.16 mm to (84.9, 82.7)
- moved D3 0.16 mm to (68.3, 82.9)
- moved D4 0.16 mm to (79.2, 82.9)
- moved Q3 0.16 mm to (50.2, 90.2)
- moved R49 0.16 mm to (66.2, 82.9)
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Connections:
- new net DAC_NRST: IC13.28, IC7.14
- new net N$51: Q10.2, R33.2
- new net N$56: D5.2, Q3.1, R34.2, R51.1
- new net N$57: Q7.2, R45.2
- new net N$58: Q8.2, R46.1
- net N$16: now also R45.1; no longer Q7.2
- net N$29: now also R34.1; no longer D5.2, Q3.1, R51.1
- net N$49: now also R46.2; no longer Q8.2
- net N$54: now also R33.1; no longer Q10.2
Routing:
- net DAC_NRST: track 0.00 -> 30.9 mm, vias 0 -> 2
- net N$56: track 0.00 -> 22.0 mm, vias 0 -> 2
- net N$29: track 22.3 -> 2.15 mm, vias 2 -> 0
- net DAC_VCC: track 68.9 -> 60.9 mm
- net +12V: track 36.1 -> 41.1 mm
- net CLK_VDD: track 33.0 -> 29.5 mm
- net N$26: track 25.9 -> 28.3 mm
- net N$57: track 0.00 -> 2.29 mm
- net N$58: track 0.00 -> 2.15 mm
- net N$51: track 0.00 -> 1.90 mm
- net N$53: track 51.8 -> 53.4 mm
- net N$54: track 11.4 -> 10.6 mm
- net I2C_SCL: track 34.7 -> 34.1 mm
- net GND: track 91.5 -> 92.1 mm
- net DAC_VDD: track 32.3 -> 32.9 mm
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
Commit message: fix PCM1795
Parts:
- C15: value 10u -> 2.2u
- C18: value 0.1u -> 1000p
- C4, C5: value 22p -> 10p
- C40, C42: device my_rcl:1608 -> my_rcl:2012
- IC7: device my_ic:TSSOP28 -> my_ic:PCM1795
- moved C48 1.27 mm to (4.13, 58.4)
- moved C40 1.21 mm to (8.89, 58.4)
- moved C53 1.02 mm to (16.8, 49.5)
- moved R3 1.00 mm to (33.5, 25.6)
- moved C8 0.95 mm to (33.5, 23.7)
- moved C7 0.90 mm to (30.0, 25.4)
- moved C45 0.71 mm to (13.5, 62.7)
- moved R17 0.71 mm to (17.3, 62.7)
- moved IC7 0.64 mm to (15.4, 55.9)
- moved C42 0.57 mm to (21.9, 58.4)
- moved C47 0.48 mm to (11.4, 67.6)
- moved R36 0.48 mm to (15.4, 46.4)
- moved X2 0.32 mm to (10.3, 44.6)
- moved X3 0.32 mm to (19.8, 44.6)
- moved C43 0.16 mm to (15.4, 42.9)
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Connections:
- net DAC_MCLK/2: now also IC3.2; no longer IC3.3
- net GND: now also IC3.3; no longer IC3.2
Routing:
- net DAC_VCC: track 60.9 -> 28.4 mm, vias 0 -> 2
- net DAC_VDD: track 32.9 -> 37.5 mm
- net GND: track 92.1 -> 94.4 mm, vias 121 -> 120
- net DAC_MCLK/2: track 6.08 -> 4.23 mm
- net N$14: track 11.5 -> 9.87 mm
- net N$5: track 4.82 -> 6.02 mm
- net +3V3D: track 55.8 -> 56.9 mm
- net DAC_DATA: track 26.6 -> 25.7 mm
- net DAC_SCK: track 29.6 -> 28.7 mm
- net DAC_LRCLK: track 24.3 -> 23.4 mm
- net IOUTL-: track 15.2 -> 14.4 mm
- net DAC_MCLK: track 30.5 -> 29.8 mm
- net I2C_SCL: track 34.1 -> 34.8 mm
- net IOUTR+: track 14.7 -> 15.3 mm
- net N$37: track 9.90 -> 9.23 mm
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Other:
- board text added: "Audio DAC v8.1"
- board text removed: "Audio DAC v8"

Commit message: 微修正
Parts:
- added R47, R48: 10, my_rcl:2012
- moved R33 0.32 mm to (51.8, 79.4)
Connections:
- net AMP_LOUT: now also R47.1
- net AMP_ROUT: now also R48.1
- net N$33: now also R48.2
- net N$34: now also R47.2
Routing:
- net AMP_LOUT: track 62.3 -> 65.0 mm
- net AMP_ROUT: track 49.6 -> 52.3 mm
- net N$34: track 37.7 -> 40.2 mm
- net N$33: track 34.1 -> 35.8 mm
- net N$26: track 28.3 -> 28.9 mm
