File: Audio-DAC.sch (EAGLE design)
At the start: 62 parts, among them CON1 USB-5075BR-04-WH, IC1 3.3V 200mA, IC2 AT32UC3A3256, IC3 OCT_BUFFER-SO6, IC4 OCT_BUFFER-SO6, IC5 OCT_BUFFER-SO6, IC6 OCT_BUFFER-SO6, IC7 OCT_BUFFER-SO6, X1 12MHz

Commit message: アイソレーター追加
Parts:
- added C25, C27, C31, C34, C38, C41, C42, C44, C45: 0.1u, my_rcl:C-1608
- added C26: 10u, my_rcl:C-1608
- added C28, C29, C35, C36: 1000u, my_rcl:CPOLE5-13
- added C30: 22u, my_rcl:C-2012
- added C32, C33: 1000u, my_rcl:CPOLE5-10
- added C37, C43, C70: 10u, my_rcl:C-2012
- added C39, C47, C59: 220u, my_rcl:CPOLE2.5-8
- added C40, C46, C52, C54, C58: 100u, my_rcl:CPOLE2.5-6.5
- added C48, C49, C53, C55: 0.22u, my_rcl:C-1608
- added C50, C51, C56, C57: DNP, my_rcl:C-1608
- added C60, C61: 100u, my_rcl:CPOLE2.5-8
- added C62, C63, C64, C65: 2000p, my_rcl:C-1608
- added C66, C67, C68, C69: 1000p, my_rcl:C-1608
- added D3, D4, D5, D6: 1N4148, my_rcl:DIODE-2
- added D7, D8: SBD-1A, my_rcl:SBD-1A
- added DR1, DR2, DR3, DR4: HOLE-3.2, my_connector:HOLE-3.2
- added FB1, FB2: FB-1608, my_rcl:FB-1608
- added IC10: -15V, my_ic:79X-LED
- added IC11: 3.3V, my_ic:NJM2863
- added IC12: LPC1114FDH28, my_ic:LPC1114FDH28
- added IC13: 7812, my_ic:78X-1
- added IC14, IC15: 5V, my_ic:78X-LED
- added IC16: 3.3V, my_ic:78X-LED
- added IC17: TC7WH74FU, my_ic:TC7WH74FU
- added IC18: AK4495EQ, my_ic:AK4495EQ
- added IC19: TC7WU04FU, my_ic:TC7WU04FU
- added IC20: 9V, my_ic:78X-LED
- added IC21: -9V, my_ic:79X-LED
- added IC22: OP275, my_ic:OPA-2'
- added IC8: 7805, my_ic:78X-SOP
- added IC9: 15V, my_ic:78X-LED
- added JP1: VOL, pinhead:PINHD-1X3
- added JP2: SWD, pinhead:PINHD-1X5
- added JP3: SPK, pinhead:PINHD-1X4
- added JP4: HP, pinhead:PINHD-1X4
- added L1, L2: 1u, my_rcl:L-7
- added Q1, Q3: NPN2SC3422, my_ic:NPN2SC3422
- added Q2, Q4: PNP2SA1359, my_ic:PNP2SA1359
- added Q5, Q6: NPN2SC3325, my_ic:NPN2SC3325
- added R24, R25: 1, my_rcl:R-10
- added R26, R27, R28, R55, R57: 10k, my_rcl:R-1608
- added R29, R30, R31: 100, my_rcl:R-5
- added R32, R33: 37, my_rcl:R-1608
- added R34, R35, R36, R37, R42, R43, R44, R45, R46, R47, R48, R49: 1k, my_rcl:R-2.5
- added R38, R39, R40, R41: 2k, my_rcl:R-2.5
- added R50, R51, R52, R53: 1, my_rcl:R-2.5
- added R54, R56: 1.5k, my_rcl:R-1608
- added SW1, SW2: EA2, my_rcl:EA2
- added TP10: TEST_2, my_connector:TESTPIN
- added TP11: TEST_4, my_connector:TESTPIN
- added TP12: TEST_6, my_connector:TESTPIN
- added TP13, TP17, TP21: GND, my_connector:TESTPIN
- added TP14: +3V3, my_connector:TESTPIN
- added TP15, TP18: SP_SW, my_connector:TESTPIN
- added TP16, TP19: HP_SW, my_connector:TESTPIN
- added TP20, TP22: +12V, my_connector:TESTPIN
- added TP5: VIN+, my_connector:TESTPIN-BIG
- added TP6, TP7: GND, my_connector:TESTPIN-BIG
- added TP8: VIN-, my_connector:TESTPIN-BIG
- added TP9: TEST_1, my_connector:TESTPIN
- added X2: 22.5792MHz, my_rcl:OSC-KC7050
- added X3: 24.576MHz, my_rcl:OSC-KC7050
- C15: value 10u -> 0.1u; device my_rcl:C-2012 -> my_rcl:C-1608
- C16: value 0.1u -> 10u; device my_rcl:C-1608 -> my_rcl:C-2012
- C3: value 22u -> 10u
- C4: value 22p -> 22u; device my_rcl:C-1608 -> my_rcl:C-2012
- C6: value 0.1u -> 22p
- C8: value 10p -> 0.1u
- C9: value 0.1u -> 10p
Connections:
- removed net AGND: C21.2, C22.2, C23.2, C24.2, IC3.C, IC4.GND, IC5.GND, IC6.GND, IC7.GND, R22.1
- new net +12V: C39.1, C70.1, D7.K, D8.K, IC13.OUT, IC14.IN, IC15.IN, IC16.IN, SW1.L1, SW2.L2, TP20.1, TP22.1
- new net DAC_!EN_48K: IC19G$1.P$2, X2.EN
- new net DAC_AVDD: C40.1, C44.1, C45.1, C48.1, FB2.1, IC16.OUT, IC18.AVDD, IC18.DEM0, IC18.I2C, X2.VCC, X3.VCC
- new net DAC_DVDD: C43.1, C49.1, FB2.2, IC18.DVSS
- new net DAC_LN: IC18.OUTLN, R37.1
- new net DAC_LP: IC18.OUTLP, R36.1
- new net DAC_MCLK: IC17G$1.CK, IC18.MCLK, R32.2, R33.2
- new net DAC_PDN: IC12.DP28, IC18.PDN, R27.2
- new net DAC_RN: IC18.OUTRN, R35.1
- new net DAC_RP: IC18.OUTRP, R34.1
- new net DAC_VCC: C52.1, C53.1, C54.1, C55.1, IC14.OUT, IC18.VDDL1, IC18.VDDL2, IC18.VDDR1, IC18.VDDR2
- new net DAC_VREF: C47.1, C51.2, C57.2, C59.1, IC15.OUT, IC18.VREFHL1, IC18.VREFHL2, IC18.VREFHR1, IC18.VREFHR2
- new net GND: C22.2, C23.2, C24.2, C25.2, C26.2, C27.2, C28.2, C29.1, C30.2, C31.2, C32.2, C33.1, C34.2, C35.2, C36.1, C37.2, C38.1, C39.2, C40.2, C41.2, C42.2, C43.2, C44.2, C45.2, C46.2, C47.2, C48.2, C49.2, C50.2, C51.1, C52.2, C53.2, C54.2, C55.2, C56.2, C57.1, C58.2, C59.2, C60.2, C61.1, C62.2, C63.2, C64.2, C65.2, C67.2, C69.2, C70.2, IC10.GND, IC11.GND, IC12.AGND, IC12.GND, IC13.GND, IC14.GND, IC15.GND, IC16.GND, IC17G$2.V-, IC18.ACKS/CAD1, IC18.AVSS, IC18.DEM1, IC18.DIF2/CAD0, IC18.DVDD, IC18.NC, IC18.PSN, IC18.SMUTE/CSN, IC18.SSLOW, IC18.VREFLL1, IC18.VREFLL2, IC18.VREFLR1, IC18.VREFLR2, IC18.VSSL1, IC18.VSSL2, IC18.VSSR1, IC18.VSSR2, IC19G$2.P$1, IC19G$3.P$1, IC19G$4.V-, IC20.GND, IC21.GND, IC3.C, IC4.GND, IC5.GND, IC6.GND, IC7.GND, IC8.GND, IC9.GND, JP1.1, JP2.3, JP3.1, JP3.4, JP4.1, JP4.4, Q5.E, Q6.E, R22.1, R27.1, R39.1, R41.1, R55.1, R57.1, TP13.1, TP17.1, TP21.1, TP6.1, TP7.1, X2.GND, X3.GND
- new net HP_L: JP4.2, SW2.COM1
- new net HP_R: JP4.3, SW2.COM2
- new net HP_SW: IC12.DP17, R56.2, TP16.1, TP19.1
- new net I2C_SCL: IC12.I2C_SCI/DP27, IC18.SD/SCL, R28.1
- new net I2C_SDA: IC12.DP5/SDA_I2C, IC18.SLOW/SDA, R26.1
- new net N$20: C69.1, IC22G$1.+IN, R45.2
- new net N$21: C66.2, IC22G$2.-IN, R42.2
- new net N$22: C67.1, IC22G$2.+IN, R43.2
- new net N$23: C68.2, IC22G$1.-IN, R44.2
- new net N$24: C66.1, L2.1, R38.2, R52.1, R53.2
- new net N$25: Q3.E, R52.2
- new net N$26: D5.A, Q3.B, R48.1
- new net N$27: D5.K, D6.A, IC22G$2.OUT
- new net N$28: Q4.E, R53.1
- new net N$29: D6.K, Q4.B, R49.2
- new net N$30: Q2.E, R51.1
- new net N$31: Q1.E, R50.2
- new net N$32: C68.1, L1.1, R40.2, R50.1, R51.2
- new net N$33: L2.2, SW1.A1, SW2.A2
- new net N$34: L1.2, SW1.A2, SW2.A1
- new net N$35: Q5.B, R54.1, R55.2
- new net N$36: D7.A, Q5.C, SW1.L2
- new net N$37: C28.1, IC9.IN, R24.2
- new net N$38: C29.2, IC10.IN, R25.2
- new net N$39: R24.1, TP5.1
- new net N$40: R25.1, TP8.1
- new net N$41: IC18.BCK, R29.2
- new net N$42: IC18.LRCK, R31.2
- new net N$43: IC18.SDATA, R30.2
- new net N$44: C64.1, R36.2, R40.1, R44.1
- new net N$45: C65.1, R37.2, R41.2, R45.1
- new net N$46: C62.1, R34.2, R38.1, R42.1
- new net N$47: C63.1, R35.2, R39.2, R43.1
- new net N$48: Q6.B, R56.1, R57.2
- new net N$49: D8.A, Q6.C, SW2.L1
- new net N$50: C34.1, IC11.BYPASS
- new net N$51: C30.1, IC11.CONTROL, IC11.VIN, IC8.OUT
- new net N$52: C27.1, IC12.DP13/AN, JP1.2
- new net N$60: D3.A, Q1.B, R46.1
- new net N$64: D4.K, Q2.B, R47.2
- new net N$75: D3.K, D4.A, IC22G$1.OUT
- new net N$83: R32.1, X2.OUT
- new net N$86: R33.1, X3.OUT
- new net N$90: IC17G$1.!Q, IC17G$1.D
- new net N$94: IC12.SWCLK, JP2.1
- new net N$95: IC12.NR/DP23, JP2.2
- new net N$96: IC12.SWDIO, JP2.4
- new net N$97: IC12.SERIAL_TX/DP16, JP2.5
- new net OPA_+: C60.1, IC20.OUT, IC22G$3.V+
- new net OPA_-: C61.2, IC21.OUT, IC22G$3.V-
- new net SPK_L: JP3.2, SW1.COM2
- new net SPK_R: JP3.3, SW1.COM1
- new net SP_SW: IC12.PWM/DP18, R54.2, TP15.1, TP18.1
- new net TEST_1: IC12.DP1/MISO_SPI/PWM, TP9.1
- new net TEST_2: IC12.DP2/MOSI_SPI/PWM, TP10.1
- new net TEST_4: IC12.DP4/AN, TP11.1
- new net TEST_6: IC12.DP6/SCK_SPI, TP12.1
- new net V+: C26.1, C32.1, C35.1, IC13.IN, IC20.IN, IC8.IN, IC9.OUT, Q1.C, Q3.C, R46.2, R48.2
- new net V-: C33.2, C36.2, IC10.OUT, IC21.IN, Q2.C, Q4.C, R47.1, R49.1
- new net VBUS: CON1.VBUS, FB1.1
- new net VCOM_L: C46.1, C50.1, IC18.VCOML
- new net VCOM_R: C56.1, C58.1, IC18.VCOMR
- net +3V3: now also C25.1, C31.1, C37.1, C38.2, C41.1, C42.1, IC11.VOUT, IC12.AVIN, IC12.VIN, IC17G$1.!CLR, IC17G$1.!PR, IC17G$2.V+, IC19G$4.V+, JP1.3, R26.2, R28.2, TP14.1; no longer C21.1
- net +3V3D: now also C11.2, C12.1, C14.1, C15.2, C17.2, C18.1, C21.1, C4.1, C8.1; no longer C11.1, C13.1, C14.2, C16.2, C17.1, C19.1, C3.1, C6.1, C9.2
- net DAC_DATA: now also R30.1
- net DAC_EN_48K: now also IC19G$1.P$1, X3.EN
- net DAC_LRCLK: now also R31.1
- net DAC_MCLK/2: now also IC17G$1.Q
- net DAC_SCK: now also R29.1
- net DGND: now also C11.1, C14.2, C17.1, C18.2, C19.1, C21.2, C9.2; no longer C11.2, C14.1, C17.2, C18.1, C19.2, C9.1
- net D_!RST: now also C13.1; no longer C12.1
- net N$3: now also C6.1; no longer C5.1
- net N$4: now also C5.1; no longer C4.1
- net N$5: now also C9.1; no longer C8.1
- net N$8: now also C16.2, C19.2; no longer C15.2, C18.2
- net USB_VBUS: now also C3.1, FB1.2; no longer CON1.VBUS

Commit message: デジタル部配置
Parts:
- removed C1: 22u, my_rcl:C-2012
- R29, R30, R31: device my_rcl:R-5 -> my_rcl:R-1608
Connections:
- net DGND: no longer C1.2
- net USB_VBUS: no longer C1.1
Changed lines of the file:
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@@
 <part name="C2" library="my_rcl" deviceset="C" device="-1608" value="0.1u"/>
 <part name="C4" library="my_rcl" deviceset="C" device="-2012" value="22u"/>
-<part name="C1" library="my_rcl" deviceset="C" device="-2012" value="22u"/>
 <part name="SUPPLY44" library="my_supply" deviceset="DGND" device=""/>
 <part name="SUPPLY45" library="my_supply" deviceset="DGND" device=""/>
@@
 <part name="R24" library="my_rcl" deviceset="R" device="-10" value="1"/>
 <part name="R25" library="my_rcl" deviceset="R" device="-10" value="1"/>
-<part name="R29" library="my_rcl" deviceset="R" device="-5" value="100"/>
-<part name="R31" library="my_rcl" deviceset="R" device="-5" value="100"/>
-<part name="R30" library="my_rcl" deviceset="R" device="-5" value="100"/>
+<part name="R29" library="my_rcl" deviceset="R" device="-1608" value="100"/>
+<part name="R31" library="my_rcl" deviceset="R" device="-1608" value="100"/>
+<part name="R30" library="my_rcl" deviceset="R" device="-1608" value="100"/>
 <part name="DR1" library="my_connector" deviceset="HOLE-3.2" device=""/>
 <part name="DR3" library="my_connector" deviceset="HOLE-3.2" device=""/>
@@
 <attribute name="VALUE" x="1.27" y="56.515" size="1.778" layer="96"/>
 </instance>
-<instance part="C1" gate="G$1" x="-35.56" y="58.42" smashed="yes" rot="MR0">
-<attribute name="NAME" x="-36.83" y="59.055" size="1.778" layer="95" rot="MR0"/>
-<attribute name="VALUE" x="-36.83" y="56.515" size="1.778" layer="96" rot="MR0"/>
-</instance>
 <instance part="SUPPLY44" gate="G$1" x="-35.56" y="53.34" smashed="yes"/>
 <instance part="SUPPLY45" gate="G$1" x="-7.62" y="50.8" smashed="yes"/>
@@
 </segment>
 <segment>
-<pinref part="C1" gate="G$1" pin="2"/>
 <pinref part="IC1" gate="G$1" pin="GND"/>
 <wire x1="-35.56" y1="55.88" x2="-33.02" y2="55.88" width="0.1524" layer="91"/>
 <pinref part="SUPPLY44" gate="G$1" pin="DGND"/>
-<junction x="-35.56" y="55.88"/>
 </segment>
 <segment>
@@
 <pinref part="IC1" gate="G$1" pin="VIN"/>
 <wire x1="-33.02" y1="60.96" x2="-33.02" y2="66.04" width="0.1524" layer="91"/>
-<wire x1="-33.02" y1="66.04" x2="-35.56" y2="66.04" width="0.1524" layer="91"/>
 <junction x="-33.02" y="66.04"/>
-<pinref part="C1" gate="G$1" pin="1"/>
-<wire x1="-35.56" y1="66.04" x2="-35.56" y2="60.96" width="0.1524" layer="91"/>
-<wire x1="-35.56" y1="66.04" x2="-38.1" y2="66.04" width="0.1524" layer="91"/>
-<junction x="-35.56" y="66.04"/>
+<wire x1="-33.02" y1="66.04" x2="-38.1" y2="66.04" width="0.1524" layer="91"/>
 <label x="-38.1" y="66.04" size="1.27" layer="95" rot="R180" xref="yes"/>
 </segment>

Commit message: 配置
Parts:
- removed C41: 0.1u, my_rcl:C-1608
- removed JP1: VOL, pinhead:PINHD-1X3
- removed JP2: SWD, pinhead:PINHD-1X5
- added CON2: SWD_CON, my_connector:SWD_CON
- added CON3: VOL_CON, my_connector:VOL_CON
- added TP23: SDA, my_connector:TESTPIN
- added TP24: SCL, my_connector:TESTPIN
- TP10: value TEST_2 -> TEST_11
- TP11: value TEST_4 -> TEST_10
- TP12: value TEST_6 -> TEST_9
- TP9: value TEST_1 -> TEST_12
Connections:
- net N$37 renamed VIN+
- net N$38 renamed VIN-
- removed net TEST_1: IC12.DP1/MISO_SPI/PWM, TP9.1
- removed net TEST_2: IC12.DP2/MOSI_SPI/PWM, TP10.1
- removed net TEST_4: IC12.DP4/AN, TP11.1
- removed net TEST_6: IC12.DP6/SCK_SPI, TP12.1
- new net N$37: IC12.DP14, TP9.1
- new net N$38: IC12.DP11/AN, TP10.1
- new net N$53: IC12.DP10/AN, TP11.1
- new net N$54: IC12.DP9/AN, TP12.1
- net +12V: now also C26.1, IC8.IN
- net +3V3: now also CON3.VCC, IC19G$2.P$1; no longer C41.1, JP1.3
- net GND: now also CON2.GND, CON3.GND; no longer C41.2, IC19G$2.P$1, JP1.1, JP2.3
- net I2C_SCL: now also TP24.1
- net I2C_SDA: now also TP23.1
- net N$52: now also CON3.VOL; no longer JP1.2
- net N$94: now also CON2.SWCLK; no longer JP2.1
- net N$95: now also CON2.!RST; no longer JP2.2
- net N$96: now also CON2.SWDIO; no longer JP2.4
- net N$97: now also CON2.TX; no longer JP2.5
- net V+: no longer C26.1, IC8.IN

Commit message: べた以外できた
Parts:
- added C1, C41: 0.1u, my_rcl:C-1608
Connections:
- net GND: now also C1.2, C41.1
- net OPA_+: now also C1.1
- net OPA_-: now also C41.2
Other:
- moved on the sheet: IC22G$3
Changed lines of the file:
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@@
 <part name="TP23" library="my_connector" deviceset="TESTPIN" device="" value="SDA"/>
 <part name="TP24" library="my_connector" deviceset="TESTPIN" device="" value="SCL"/>
+<part name="C1" library="my_rcl" deviceset="C" device="-1608" value="0.1u"/>
+<part name="C41" library="my_rcl" deviceset="C" device="-1608" value="0.1u"/>
 </parts>
 <sheets>
@@
 <attribute name="VALUE" x="94.234" y="160.147" size="1.778" layer="96"/>
 </instance>
-<instance part="SUPPLY82" gate="GND" x="101.6" y="165.1" smashed="yes"/>
+<instance part="SUPPLY82" gate="GND" x="109.22" y="165.1" smashed="yes"/>
 <instance part="IC20" gate="G$1" x="78.74" y="180.34" smashed="yes">
 <attribute name="NAME" x="76.2" y="182.88" size="1.778" layer="95"/>
@@
 </instance>
 <instance part="SUPPLY83" gate="GND" x="83.82" y="165.1" smashed="yes"/>
-<instance part="IC22" gate="G$3" x="109.22" y="170.18" smashed="yes">
-<attribute name="NAME" x="111.76" y="175.26" size="1.778" layer="95"/>
+<instance part="IC22" gate="G$3" x="114.3" y="170.18" smashed="yes">
+<attribute name="NAME" x="116.84" y="175.26" size="1.778" layer="95"/>
 </instance>
 <instance part="C40" gate="G$1" x="-60.96" y="99.06" smashed="yes" rot="MR0">
@@
 <instance part="TP24" gate="G$1" x="-78.74" y="-30.48" smashed="yes" rot="R270">
 <attribute name="VALUE" x="-74.295" y="-31.115" size="1.778" layer="95"/>
+</instance>
+<instance part="C1" gate="G$1" x="101.6" y="175.26" smashed="yes">
+<attribute name="NAME" x="102.87" y="175.895" size="1.778" layer="95"/>
+<attribute name="VALUE" x="102.87" y="173.355" size="1.778" layer="96"/>
+</instance>
+<instance part="C41" gate="G$1" x="101.6" y="162.56" smashed="yes">
+<attribute name="NAME" x="102.87" y="163.195" size="1.778" layer="95"/>
+<attribute name="VALUE" x="102.87" y="160.655" size="1.778" layer="96"/>
 </instance>
 </instances>
@@
 <junction x="93.98" y="170.18"/>
 <pinref part="SUPPLY82" gate="GND" pin="GND"/>
-<wire x1="101.6" y1="170.18" x2="101.6" y2="167.64" width="0.1524" layer="91"/>
+<wire x1="101.6" y1="170.18" x2="109.22" y2="170.18" width="0.1524" layer="91"/>
+<wire x1="109.22" y1="170.18" x2="109.22" y2="167.64" width="0.1524" layer="91"/>
+<pinref part="C1" gate="G$1" pin="2"/>
+<wire x1="101.6" y1="172.72" x2="101.6" y2="170.18" width="0.1524" layer="91"/>
+<junction x="101.6" y="170.18"/>
+<pinref part="C41" gate="G$1" pin="1"/>
+<wire x1="101.6" y1="170.18" x2="101.6" y2="165.1" width="0.1524" layer="91"/>
 </segment>
 <segment>
@@
 <pinref part="IC21" gate="G$1" pin="OUT"/>
 <pinref part="C61" gate="G$1" pin="2"/>
-<wire x1="109.22" y1="157.48" x2="93.98" y2="157.48" width="0.1524" layer="91"/>
+<wire x1="114.3" y1="157.48" x2="101.6" y2="157.48" width="0.1524" layer="91"/>
+<wire x1="101.6" y1="157.48" x2="93.98" y2="157.48" width="0.1524" layer="91"/>
 <wire x1="93.98" y1="157.48" x2="88.9" y2="157.48" width="0.1524" layer="91"/>
 <wire x1="93.98" y1="160.02" x2="93.98" y2="157.48" width="0.1524" layer="91"/>
 <junction x="93.98" y="157.48"/>
 <pinref part="IC22" gate="G$3" pin="V-"/>
-<wire x1="109.22" y1="162.56" x2="109.22" y2="157.48" width="0.1524" layer="91"/>
+<wire x1="114.3" y1="162.56" x2="114.3" y2="157.48" width="0.1524" layer="91"/>
 <label x="93.98" y="157.48" size="1.778" layer="95" rot="R270" xref="yes"/>
+<pinref part="C41" gate="G$1" pin="2"/>
+<wire x1="101.6" y1="160.02" x2="101.6" y2="157.48" width="0.1524" layer="91"/>
+<junction x="101.6" y="157.48"/>
 </segment>
 </net>
@@
 <pinref part="IC20" gate="G$1" pin="OUT"/>
 <pinref part="IC22" gate="G$3" pin="V+"/>
-<wire x1="109.22" y1="180.34" x2="93.98" y2="180.34" width="0.1524" layer="91"/>
+<wire x1="114.3" y1="180.34" x2="101.6" y2="180.34" width="0.1524" layer="91"/>
+<wire x1="101.6" y1="180.34" x2="93.98" y2="180.34" width="0.1524" layer="91"/>
 <wire x1="93.98" y1="180.34" x2="88.9" y2="180.34" width="0.1524" layer="91"/>
-<wire x1="109.22" y1="180.34" x2="109.22" y2="177.8" width="0.1524" layer="91"/>
+<wire x1="114.3" y1="180.34" x2="114.3" y2="177.8" width="0.1524" layer="91"/>
 <pinref part="C60" gate="G$1" pin="1"/>
 <wire x1="93.98" y1="180.34" x2="93.98" y2="177.8" width="0.1524" layer="91"/>
 <junction x="93.98" y="180.34"/>
 <label x="93.98" y="180.34" size="1.778" layer="95" rot="R90" xref="yes"/>
-</segment>
-</net>
+<pinref part="C1" gate="G$1" pin="1"/>
+<wire x1="101.6" y1="180.34" x2="101.6" y2="177.8" width="0.1524" layer="91"/>
+<junction x="101.6" y="180.34"/>
+</segment>
+</net>

Commit message: DDCのフォトカプラ追加
Parts:
- added C71: 10u, my_rcl:C-2012
- added DECO1: ROBOTECH_WHEEL, my_connector:ROBOTECH_WHEEL
- added IC23: OP275, my_ic:OPA-2'
- added R58, R60: 10k, my_rcl:R-1608
- added R59: 1.5k, my_rcl:R-1608
- C15, C2, C42: value 0.1u -> 10u; device my_rcl:C-1608 -> my_rcl:C-2012
- C16, C43: value 10u -> 0.1u; device my_rcl:C-2012 -> my_rcl:C-1608
- C3: value 10u -> 22u
- C4: value 22u -> 22p; device my_rcl:C-2012 -> my_rcl:C-1608
- C45: value 0.1u -> 100u; device my_rcl:C-1608 -> my_rcl:CPOLE2.5-6.5
- C46, C58: value 100u -> 220u; device my_rcl:CPOLE2.5-6.5 -> my_rcl:CPOLE2.5-8
- C47: value 220u -> 0.22u; device my_rcl:CPOLE2.5-8 -> my_rcl:C-1608
- C49, C55: value 0.22u -> DNP
- C51, C57: value DNP -> 100u; device my_rcl:C-1608 -> my_rcl:CPOLE2.5-6.5
- C52, C54: value 100u -> 0.22u; device my_rcl:CPOLE2.5-6.5 -> my_rcl:C-1608
- C53: value 0.22u -> 100u; device my_rcl:C-1608 -> my_rcl:CPOLE2.5-6.5
- C59: value 220u -> 100u
- C6: value 22p -> 0.1u
- C61: value 100u -> 0.1u; device my_rcl:CPOLE2.5-8 -> my_rcl:C-1608
- C62: value 2000p -> 0.1u
- C66: value 1000p -> 2000p
- C70: value 10u -> 1000p; device my_rcl:C-2012 -> my_rcl:C-1608
- C8: value 0.1u -> 10p
- C9: value 10p -> 0.1u
- CON2: value SWD_CON -> VOL_CON; device my_connector:SWD_CON -> my_connector:VOL_CON
- CON3: value VOL_CON -> SWD_CON; device my_connector:VOL_CON -> my_connector:SWD_CON
- IC10: value -15V -> 15V; device my_ic:79X-LED -> my_ic:78X-LED
- IC11: value 3.3V -> -15V; device my_ic:NJM2863 -> my_ic:79X-LED
- IC12: value LPC1114FDH28 -> 3.3V; device my_ic:LPC1114FDH28 -> my_ic:NJM2863
- IC13: value 7812 -> LPC1114FDH28; device my_ic:78X-1 -> my_ic:LPC1114FDH28
- IC14: value 5V -> 7812; device my_ic:78X-LED -> my_ic:78X-1
- IC16: value 3.3V -> 5V
- IC17: value TC7WH74FU -> 3.3V; device my_ic:TC7WH74FU -> my_ic:78X-LED
- IC18: value AK4495EQ -> TC7WH74FU; device my_ic:AK4495EQ -> my_ic:TC7WH74FU
- IC19: value TC7WU04FU -> AK4495EQ; device my_ic:TC7WU04FU -> my_ic:AK4495EQ
- IC20: value 9V -> TC7WU04FU; device my_ic:78X-LED -> my_ic:TC7WU04FU
- IC21: value -9V -> 9V; device my_ic:79X-LED -> my_ic:78X-LED
- IC22: value OP275 -> -9V; device my_ic:OPA-2' -> my_ic:79X-LED
- IC8: value 7805 -> OCT_BUFFER-SO6; device my_ic:78X-SOP -> my_ic:OCT_BUFFER-SO6
- IC9: value 15V -> 7805; device my_ic:78X-LED -> my_ic:78X-SOP
- R23: value 1.5k -> 10k
- R24: value 1 -> 10k; device my_rcl:R-10 -> my_rcl:R-1608
- R25: value 1 -> 1.5k; device my_rcl:R-10 -> my_rcl:R-1608
- R26, R57: value 10k -> 1.5k
- R27, R28: value 10k -> 1; device my_rcl:R-1608 -> my_rcl:R-10
- R29, R30, R31: value 100 -> 10k
- R32, R33: value 37 -> 100
- R34: value 1k -> 100; device my_rcl:R-2.5 -> my_rcl:R-1608
- R35, R36: value 1k -> 37; device my_rcl:R-2.5 -> my_rcl:R-1608
- R38, R39, R40: value 2k -> 1k
- R4, R5: value 33 -> 39
- R42, R43, R44: value 1k -> 2k
- R50, R51, R52: value 1 -> 1k
- R54, R56: value 1.5k -> 1; device my_rcl:R-1608 -> my_rcl:R-2.5
- R55: value 10k -> 1; device my_rcl:R-1608 -> my_rcl:R-2.5
- renumbered JP3 to JP1, JP4 to JP2
Connections:
- new net EN_+3V3D: IC1.CONTROL, IC8.OUT, R18.2
- new net EN_DDC: IC13.DP1/MISO_SPI/PWM, R26.1
- new net N$55: IC8.A, R24.2, R26.2
- net +12V: now also C71.1, IC14.OUT, IC17.IN, IC9.IN; no longer C70.1, IC13.OUT, IC14.IN, IC8.IN
- net +3V3: now also C41.1, CON2.VCC, IC12.VOUT, IC13.AVIN, IC13.VIN, IC18G$1.!CLR, IC18G$1.!PR, IC18G$2.V+, IC20G$2.P$1, IC20G$4.V+, R29.2, R31.2; no longer C42.1, CON3.VCC, IC11.VOUT, IC12.AVIN, IC12.VIN, IC17G$1.!CLR, IC17G$1.!PR, IC17G$2.V+, IC19G$2.P$1, IC19G$4.V+, R26.2, R28.2
- net +3V3D: now also C11.1, C13.1, C14.2, C16.2, C17.1, C19.1, C3.1, C6.1, C9.2; no longer C11.2, C12.1, C14.1, C15.2, C17.2, C18.1, C20.1, C4.1, C8.1
- net DAC_!EN_48K: now also IC20G$1.P$2; no longer IC19G$1.P$2
- net DAC_AVDD: now also C43.1, C47.1, IC17.OUT, IC19.AVDD, IC19.DEM0, IC19.I2C; no longer C45.1, C48.1, IC16.OUT, IC18.AVDD, IC18.DEM0, IC18.I2C
- net DAC_DATA: now also R33.1; no longer R30.1
- net DAC_DVDD: now also C42.1, C48.1, IC19.DVSS; no longer C43.1, C49.1, IC18.DVSS
- net DAC_EN_48K: now also IC20G$1.P$1; no longer IC19G$1.P$1
- net DAC_LN: now also IC19.OUTLN, R40.1; no longer IC18.OUTLN, R37.1
- net DAC_LP: now also IC19.OUTLP, R39.1; no longer IC18.OUTLP, R36.1
- net DAC_LRCLK: now also R34.1; no longer R31.1
- net DAC_MCLK: now also IC18G$1.CK, IC19.MCLK, R35.2, R36.2; no longer IC17G$1.CK, IC18.MCLK, R32.2, R33.2
- net DAC_MCLK/2: now also IC18G$1.Q, R25.1; no longer IC17G$1.Q, R23.1
- net DAC_PDN: now also IC13.DP28, IC19.PDN, R30.2; no longer IC12.DP28, IC18.PDN, R27.2
- net DAC_RN: now also IC19.OUTRN, R38.1; no longer IC18.OUTRN, R35.1
- net DAC_RP: now also IC19.OUTRP, R37.1; no longer IC18.OUTRP, R34.1
- net DAC_SCK: now also R32.1; no longer R29.1
- net DAC_VCC: now also C51.1, IC15.OUT, IC19.VDDL1, IC19.VDDL2, IC19.VDDR1, IC19.VDDR2; no longer C55.1, IC14.OUT, IC18.VDDL1, IC18.VDDL2, IC18.VDDR1, IC18.VDDR2
- net DAC_VREF: now also C46.1, C50.2, C56.2, C58.1, IC16.OUT, IC19.VREFHL1, IC19.VREFHL2, IC19.VREFHR1, IC19.VREFHR2; no longer C47.1, C51.2, C57.2, C59.1, IC15.OUT, IC18.VREFHL1, IC18.VREFHL2, IC18.VREFHR1, IC18.VREFHR2
- net DGND: now also C1.2, C11.2, C14.1, C17.2, C18.1, C19.2, C9.1, IC8.GND, R22.1; no longer C11.1, C14.2, C17.1, C18.2, C19.1, C9.2
- net D_!RST: now also C12.1; no longer C13.1
- net GND: now also C41.2, C50.1, C51.2, C56.1, C57.2, C60.1, C61.2, C62.1, C66.2, C68.2, C71.2, IC13.AGND, IC17.GND, IC18G$2.V-, IC19.ACKS/CAD1, IC19.AVSS, IC19.DEM1, IC19.DIF2/CAD0, IC19.DVDD, IC19.NC, IC19.PSN, IC19.SMUTE/CSN, IC19.SSLOW, IC19.VREFLL1, IC19.VREFLL2, IC19.VREFLR1, IC19.VREFLR2, IC19.VSSL1, IC19.VSSL2, IC19.VSSR1, IC19.VSSR2, IC20G$3.P$1, IC20G$4.V-, IC22.GND, IC8.C, R23.1, R24.1, R30.1, R42.1, R44.1, R58.1, R60.1; no longer C1.2, C41.1, C50.2, C51.1, C56.2, C57.1, C60.2, C61.1, C62.2, C67.2, C69.2, IC12.AGND, IC17G$2.V-, IC18.ACKS/CAD1, IC18.AVSS, IC18.DEM1, IC18.DIF2/CAD0, IC18.DVDD, IC18.NC, IC18.PSN, IC18.SMUTE/CSN, IC18.SSLOW, IC18.VREFLL1, IC18.VREFLL2, IC18.VREFLR1, IC18.VREFLR2, IC18.VSSL1, IC18.VSSL2, IC18.VSSR1, IC18.VSSR2, IC19G$3.P$1, IC19G$4.V-, IC20.GND, IC8.GND, R22.1, R27.1, R39.1, R41.1, R55.1, R57.1
- net HP_SW: now also IC13.DP17, R59.2; no longer IC12.DP17, R56.2
- net I2C_SCL: now also IC13.I2C_SCI/DP27, IC19.SD/SCL, R31.1; no longer IC12.I2C_SCI/DP27, IC18.SD/SCL, R28.1
- net I2C_SDA: now also IC13.DP5/SDA_I2C, IC19.SLOW/SDA, R29.1; no longer IC12.DP5/SDA_I2C, IC18.SLOW/SDA, R26.1
- net N$14: now also R22.2; no longer R21.2
- net N$15: now also R19.2; no longer R18.2
- net N$16: now also R20.2; no longer R19.2
- net N$17: now also R21.2; no longer R20.2
- net N$18: now also C1.1; no longer C2.1
- net N$19: now also R25.2; no longer R22.2
- net N$20: now also C70.1, IC23G$1.+IN, R48.2; no longer C69.1, IC22G$1.+IN, R45.2
- net N$21: now also C67.2, IC23G$2.-IN, R45.2; no longer C66.2, IC22G$2.-IN, R42.2
- net N$22: now also C68.1, IC23G$2.+IN, R46.2; no longer C67.1, IC22G$2.+IN, R43.2
- net N$23: now also C69.2, IC23G$1.-IN, R47.2; no longer C68.2, IC22G$1.-IN, R44.2
- net N$24: now also C67.1, R41.2, R55.1, R56.2; no longer C66.1, R38.2, R52.1, R53.2
- net N$25: now also R55.2; no longer R52.2
- net N$26: now also R51.1; no longer R48.1
- net N$27: now also IC23G$2.OUT; no longer IC22G$2.OUT
- net N$28: now also R56.1; no longer R53.1
- net N$29: now also R52.2; no longer R49.2
- net N$3: now also C5.1; no longer C6.1
- net N$30: now also R54.1; no longer R51.1
- net N$31: now also R53.2; no longer R50.2
- net N$32: now also C69.1, R43.2, R53.1, R54.2; no longer C68.1, R40.2, R50.1, R51.2
- net N$35: now also R57.1, R58.2; no longer R54.1, R55.2
- net N$37: now also IC13.DP14; no longer IC12.DP14
- net N$38: now also IC13.DP11/AN; no longer IC12.DP11/AN
- net N$39: now also R27.1; no longer R24.1
- net N$4: now also C4.1; no longer C5.1
- net N$40: now also R28.1; no longer R25.1
- net N$41: now also IC19.BCK, R32.2; no longer IC18.BCK, R29.2
- net N$42: now also IC19.LRCK, R34.2; no longer IC18.LRCK, R31.2
- net N$43: now also IC19.SDATA, R33.2; no longer IC18.SDATA, R30.2
- net N$44: now also C65.1, R39.2, R43.1, R47.1; no longer C64.1, R36.2, R40.1, R44.1
- net N$45: now also C66.1, R40.2, R44.2, R48.1; no longer C65.1, R37.2, R41.2, R45.1
- net N$46: now also C63.1, R37.2, R41.1, R45.1; no longer C62.1, R34.2, R38.1, R42.1
- net N$47: now also C64.1, R38.2, R42.2, R46.1; no longer C63.1, R35.2, R39.2, R43.1
- net N$48: now also R59.1, R60.2; no longer R56.1, R57.2
- net N$5: now also C8.1; no longer C9.1
- net N$50: now also IC12.BYPASS; no longer IC11.BYPASS
- net N$51: now also IC12.CONTROL, IC12.VIN, IC9.OUT; no longer IC11.CONTROL, IC11.VIN, IC8.OUT
- net N$52: now also CON2.VOL, IC13.DP13/AN; no longer CON3.VOL, IC12.DP13/AN
- net N$53: now also IC13.DP10/AN; no longer IC12.DP10/AN
- net N$54: now also IC13.DP9/AN; no longer IC12.DP9/AN
- net N$60: now also R49.1; no longer R46.1
- net N$64: now also R50.2; no longer R47.2
- net N$75: now also IC23G$1.OUT; no longer IC22G$1.OUT
- net N$8: now also C15.2, C18.2; no longer C16.2, C19.2
- net N$83: now also R35.1; no longer R32.1
- net N$86: now also R36.1; no longer R33.1
- net N$90: now also IC18G$1.!Q, IC18G$1.D; no longer IC17G$1.!Q, IC17G$1.D
- net N$94: now also CON3.SWCLK, IC13.SWCLK; no longer CON2.SWCLK, IC12.SWCLK
- net N$95: now also CON3.!RST, IC13.NR/DP23; no longer CON2.!RST, IC12.NR/DP23
- net N$96: now also CON3.SWDIO, IC13.SWDIO; no longer CON2.SWDIO, IC12.SWDIO
- net N$97: now also CON3.TX, IC13.SERIAL_TX/DP16; no longer CON2.TX, IC12.SERIAL_TX/DP16
- net OPA_+: now also C59.1, C61.1, IC21.OUT, IC23G$3.V+; no longer C1.1, C60.1, IC20.OUT, IC22G$3.V+
- net OPA_-: now also C60.2, C62.2, IC22.OUT, IC23G$3.V-; no longer C41.2, C61.2, IC21.OUT, IC22G$3.V-
- net SP_SW: now also IC13.PWM/DP18, R57.2; no longer IC12.PWM/DP18, R54.2
- net USB_VBUS: now also C2.1, C20.1, IC8.V+; no longer C3.1, IC1.CONTROL
- net V+: now also IC10.OUT, IC14.IN, IC21.IN, R49.2, R51.2; no longer IC13.IN, IC20.IN, IC9.OUT, R46.2, R48.2
- net V-: now also IC11.OUT, IC22.IN, R50.1, R52.1; no longer IC10.OUT, IC21.IN, R47.1, R49.1
- net VCOM_L: now also C45.1, C49.1, IC19.VCOML; no longer C46.1, C50.1, IC18.VCOML
- net VCOM_R: now also C55.1, C57.1, IC19.VCOMR; no longer C56.1, C58.1, IC18.VCOMR
- net VIN+: now also IC10.IN, R27.2; no longer IC9.IN, R24.2
- net VIN-: now also IC11.IN, R28.2; no longer IC10.IN, R25.2
Other:
- moved on the sheet: C10, C11, C12, C13, C14, C15, C16, C17, C18, C19, C2, C20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
