File: Audio-DAC.sch (EAGLE design)
At the start: 214 parts, among them CON1 USB-B, CON2 VOLUEME, CON3 SWD, IC1 3.3V, IC10 +15V, IC11 -15V, IC12 3.3V, IC13 LPC1114, IC14 +10V, IC15 +5V, IC17 +3.3V, IC18 TC7WH74FU, IC2 AT32UC3A3256, IC20 TC7WU04FU, IC21 +10V, IC22 -10V, IC23 OP275, IC3 SI8420, IC4 SI8420, IC5 SI8420, IC6 SI8420, IC7 PCM1795, IC9 7805, Q1 NPN-SOT223, Q10 NPN2SC3325, Q2 PNP-SOT223, Q3 NPN-SOT223, Q4 PNP-SOT223, Q5 NPN, Q6 NPN, Q7 NPN2SC3325, Q8 PNP2SA1313, Q9 PNP2SA1313, SW1 EA2, SW2 EA2, X1 12MHz, X2 24.576MHz, X3 22.5792MHz

Commit message: だいたい
Parts:
- removed C68: 1000p, my_rcl:C-1608
- removed IC12: 3.3V, my_ic:NJM2863
- removed R45, R46, R47, R48: 150, my_rcl:R-1608
- removed TP24: SCL, my_connector:TESTPIN
- added C57: 0.1u, my_rcl:C-1608
- added C58: 100u, my_rcl:CPOLE2.5-6.5
- added FB2, FB5, FB6: FB, my_rcl:FB
- added R22, R23, R24, R25: 10, my_rcl:R-1608J
- added R26, R32: 47, my_rcl:R-1608J
- added TP21: V-, my_connector:TESTPIN-BIG
- added TP22: GND, my_connector:TESTPIN-BIG
- C26: device my_rcl:C-1608 -> my_rcl:C-2012
- C30: value 22u -> 0.1u; device my_rcl:C-2012 -> my_rcl:C-1608
- C35, C36: device my_rcl:CPOLE5-13 -> my_rcl:CPOLE5-10
- C49, C50, C51, C52: value (none) -> 3300p
- C63: value 10n -> 1000p
- C64, C65, C66: value 10n -> 10u; device my_rcl:C-1608 -> my_rcl:C-2012
- IC14: value +10V -> +12V
- IC9: value 7805 -> 7803
- Q10, Q7: value NPN2SC3325 -> NPN
- Q8, Q9: value PNP2SA1313 -> PNP
- R18, R19, R20, R21: value (none) -> 1k
- R30: value 10k -> 47; device my_rcl:R-1608 -> my_rcl:R-1608J
- R37, R38, R39, R40: value 2k -> 1k
- R41, R42, R43, R44: value 4k -> 1k
- TP11: value SDA -> V+; device my_connector:TESTPIN -> my_connector:TESTPIN-BIG
Connections:
- net N$24 renamed AMP_ROUT
- net N$32 renamed AMP_LOUT
- net N$94 renamed SWCLK
- net N$95 renamed LPC_NRST
- net N$96 renamed SWDIO
- net N$97 renamed LPC_UART_TX
- removed net DAC_PDN: IC13.DP28, R30.2
- removed net N$46: C63.1, R37.2, R41.1, R45.1
- removed net N$50: C34.1, IC12.BYPASS
- removed net N$51: C30.1, IC12.CONTROL, IC12.VIN, IC9.OUT
- removed net N$56: C26.1, FB3.2, IC9.IN
- new net +12VD: C26.1, D7.K, D8.K, FB3.2, IC9.IN, SW1.L2, SW2.L2, TP15.1, TP16.1
- new net DAC_LRCLK_IN: IC5.OUT1, R15.1, R30.1
- new net N$14: C58.2, IC7.VCOMR
- new net N$24: C66.1, FB6.2, IC14.IN
- new net N$32: IC5.OUT2, R32.1
- new net N$41: C49.1, IC8G$1.-IN, R18.1, R22.2
- new net N$42: C50.1, IC8G$2.-IN, R19.1, R23.2
- new net N$43: C51.1, IC19G$1.-IN, R20.1, R24.2
- new net N$55: C52.1, IC19G$2.-IN, R21.1, R25.2
- net +12V: no longer D7.K, D8.K, SW1.L2, SW2.L2, TP15.1, TP16.1
- net +3V3: now also IC9.OUT; no longer IC12.VOUT
- net DAC_DATA: now also R32.2; no longer IC5.OUT2
- net DAC_EN_48K: no longer IC4.OUT2
- net DAC_EN_48K_IN: now also IC4.OUT2
- net DAC_LN: now also C52.2, IC19G$2.OUT, R21.2; no longer C50.2, IC8G$2.OUT, R19.2
- net DAC_LP: now also C51.2, IC19G$1.OUT, R20.2; no longer C49.2, IC8G$1.OUT, R18.2
- net DAC_LRCLK: now also R30.2; no longer IC5.OUT1, R15.1
- net DAC_MCLK: no longer IC3.IN2
- net DAC_MCLK/2: now also IC3.IN2
- net DAC_RN: now also C50.2, IC8G$2.OUT, R19.2; no longer C52.2, IC19G$2.OUT, R21.2
- net DAC_RP: now also C49.2, IC8G$1.OUT, R18.2; no longer C51.2, IC19G$1.OUT, R20.2
- net DAC_SCK: now also R26.2; no longer IC4.OUT1
- net DAC_VCC: now also C58.1; no longer C46.1
- net GND: now also C46.1, C57.1, C65.1, TP22.1; no longer C65.2, C68.2, IC12.GND, R30.1
- net I2C_SCL: no longer TP24.1
- net I2C_SDA: no longer TP11.1
- net IOUTL+: now also R25.1; no longer C49.1, IC8G$1.-IN, R18.1
- net IOUTL-: now also R24.1; no longer C50.1, C52.1, IC19G$2.-IN, IC8G$2.-IN, R19.1, R21.1
- net IOUTR+: now also R23.1; no longer C51.1, IC19G$1.-IN, R20.1
- net IOUTR-: now also R22.1
- net N$20: now also C64.1, FB2.2, IC21.IN; no longer C70.1, IC23G$1.+IN, R48.2
- net N$21: now also R37.2, R41.1; no longer R45.2
- net N$22: now also C63.1, R38.2, R42.2; no longer C68.1, R46.2
- net N$23: now also C65.2, FB5.2, IC22.IN; no longer C69.2, IC23G$1.-IN, R47.2
- net N$33: now also SW1.A2; no longer SW1.A1
- net N$34: now also SW1.A1; no longer SW1.A2
- net N$37: no longer C46.2, IC7.VCOMR
- net N$44: now also C69.2, IC23G$1.-IN; no longer C65.1, R47.1
- net N$45: now also C70.1, IC23G$1.+IN; no longer C66.1, R48.1
- net N$47: now also IC4.OUT1, R26.1; no longer C64.1, R38.2, R42.2, R46.1
- net OPA_+: now also C30.1, C34.1
- net OPA_-: now also C46.2, C57.2
- net SPK_L: now also SW1.COM1; no longer SW1.COM2
- net SPK_R: now also SW1.COM2; no longer SW1.COM1
- net V+: now also FB2.1, FB6.1, TP11.1; no longer IC14.IN, IC21.IN
- net V-: now also FB5.1, TP21.1; no longer IC22.IN
Other:
- moved on the sheet: C30, C34, C37, C46, C47, C63, C64, C65, C66, IC19G$3, IC23G$3, IC8G$3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

Commit message: 全部つないだ
Parts:
- IC23: value OP275 -> (none)
Changed lines of the file:
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@@
 <part name="SUPPLY76" library="my_supply" deviceset="GND" device=""/>
 <part name="SUPPLY77" library="my_supply" deviceset="V+" device=""/>
-<part name="IC23" library="my_ic" deviceset="OPA-2" device="-SOP" value="OP275"/>
+<part name="IC23" library="my_ic" deviceset="OPA-2" device="-SOP"/>
 <part name="R39" library="my_rcl" deviceset="R" device="-1608" value="1k"/>
 <part name="R40" library="my_rcl" deviceset="R" device="-1608" value="1k"/>
@@
 <pinref part="R30" gate="G$1" pin="1"/>
 <wire x1="274.32" y1="2.54" x2="284.48" y2="2.54" width="0.1524" layer="91"/>
-</segment>
-</net>
+<label x="273.05" y="2.54" size="1.27" layer="95"/>
+</segment>
+</net>
