File: Audio-DAC.sch (EAGLE design)
At the start: 220 parts, among them CON1 USB-B, CON2 VOLUEME, CON3 SWD, IC1 3.3V, IC10 +15V, IC11 -15V, IC13 LPC1114, IC14 +12V, IC15 +5V, IC17 +3.3V, IC18 TC7WH74FU, IC2 AT32UC3A3256, IC20 TC7WU04FU, IC21 +10V, IC22 -10V, IC3 SI8420, IC4 SI8420, IC5 SI8420, IC6 SI8420, IC7 PCM1795, IC9 7803, Q1 NPN-SOT223, Q10 NPN, Q2 PNP-SOT223, Q3 NPN-SOT223, Q4 PNP-SOT223, Q5 NPN, Q6 NPN, Q7 NPN, Q8 PNP, Q9 PNP, SW1 EA2, SW2 EA2, X1 12MHz, X2 24.576MHz, X3 22.5792MHz

Commit message: シルク整えた
Parts:
- added C68, C71: FF, my_rcl:C-1608
- TP12: value TEST_9 -> TP9
- TP13: value TEST_10 -> TP10
- TP14: value TEST_14 -> TP14
- TP23: value TEST_11 -> TP11
Connections:
- net AMP_LOUT: now also C68.1
- net AMP_ROUT: now also C71.1
- net N$26: now also C71.2
- net N$53: now also C68.2
Changed lines of the file:
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@@
 <part name="TP9" library="my_connector" deviceset="TESTPIN" device="" value="+3V3"/>
 <part name="TP10" library="my_connector" deviceset="TESTPIN" device="" value="GND"/>
-<part name="TP12" library="my_connector" deviceset="TESTPIN" device="" value="TEST_9"/>
-<part name="TP13" library="my_connector" deviceset="TESTPIN" device="" value="TEST_10"/>
-<part name="TP14" library="my_connector" deviceset="TESTPIN" device="" value="TEST_14"/>
-<part name="TP23" library="my_connector" deviceset="TESTPIN" device="" value="TEST_11"/>
+<part name="TP12" library="my_connector" deviceset="TESTPIN" device="" value="TP9"/>
+<part name="TP13" library="my_connector" deviceset="TESTPIN" device="" value="TP10"/>
+<part name="TP14" library="my_connector" deviceset="TESTPIN" device="" value="TP14"/>
+<part name="TP23" library="my_connector" deviceset="TESTPIN" device="" value="TP11"/>
 <part name="R15" library="my_rcl" deviceset="R" device="-1608J" value="100"/>
 <part name="TP27" library="my_connector" deviceset="TESTPIN" device="-BIG" value="GND_L"/>
@@
 <part name="R30" library="my_rcl" deviceset="R" device="-1608J" value="47"/>
 <part name="R32" library="my_rcl" deviceset="R" device="-1608J" value="47"/>
+<part name="C68" library="my_rcl" deviceset="C" device="-1608" value="FF"/>
+<part name="C71" library="my_rcl" deviceset="C" device="-1608" value="FF"/>
 </parts>
 <sheets>
@@
 <instance part="Q4" gate="G$1" x="276.86" y="43.18" smashed="yes">
 <attribute name="NAME" x="281.94" y="43.18" size="1.778" layer="95"/>
-<attribute name="VALUE" x="281.94" y="40.64" size="1.778" layer="96"/>
+<attribute name="VALUE" x="281.94" y="39.37" size="1.778" layer="96"/>
 </instance>
 <instance part="Q3" gate="G$1" x="276.86" y="73.66" smashed="yes">
 <attribute name="NAME" x="281.94" y="73.66" size="1.778" layer="95"/>
-<attribute name="VALUE" x="281.94" y="71.12" size="1.778" layer="96"/>
+<attribute name="VALUE" x="281.94" y="69.85" size="1.778" layer="96"/>
 </instance>
 <instance part="R55" gate="G$1" x="279.4" y="63.5" smashed="yes" rot="R90">
@@
 <instance part="Q7" gate="G$1" x="259.08" y="109.22" smashed="yes">
 <attribute name="NAME" x="255.27" y="110.49" size="1.778" layer="95"/>
-<attribute name="VALUE" x="242.57" y="106.68" size="1.778" layer="96"/>
+<attribute name="VALUE" x="252.73" y="106.68" size="1.778" layer="96"/>
 </instance>
 <instance part="Q8" gate="G$1" x="259.08" y="124.46" smashed="yes">
 <attribute name="NAME" x="254" y="125.73" size="1.778" layer="95"/>
-<attribute name="VALUE" x="243.84" y="120.65" size="1.778" layer="96"/>
+<attribute name="VALUE" x="252.73" y="120.65" size="1.778" layer="96"/>
 </instance>
 <instance part="D3" gate="G$1" x="254" y="134.62" smashed="yes" rot="R90">
@@
 <instance part="Q9" gate="G$1" x="259.08" y="66.04" smashed="yes">
 <attribute name="NAME" x="252.73" y="67.31" size="1.778" layer="95"/>
-<attribute name="VALUE" x="245.11" y="60.96" size="1.778" layer="96"/>
+<attribute name="VALUE" x="252.73" y="62.23" size="1.778" layer="96"/>
 </instance>
 <instance part="Q10" gate="G$1" x="259.08" y="50.8" smashed="yes">
 <attribute name="NAME" x="252.73" y="53.34" size="1.778" layer="95"/>
-<attribute name="VALUE" x="242.57" y="48.26" size="1.778" layer="96"/>
+<attribute name="VALUE" x="252.73" y="48.26" size="1.778" layer="96"/>
 </instance>
 <instance part="D5" gate="G$1" x="254" y="76.2" smashed="yes" rot="R90">
@@
 </instance>
 <instance part="SUPPLY103" gate="GND" x="-106.68" y="104.14" smashed="yes"/>
+<instance part="C68" gate="G$1" x="238.76" y="124.46" smashed="yes">
+<attribute name="NAME" x="240.03" y="125.095" size="1.778" layer="95"/>
+<attribute name="VALUE" x="240.03" y="122.555" size="1.778" layer="96"/>
+</instance>
+<instance part="C71" gate="G$1" x="238.76" y="66.04" smashed="yes">
+<attribute name="NAME" x="240.03" y="66.675" size="1.778" layer="95"/>
+<attribute name="VALUE" x="240.03" y="64.135" size="1.778" layer="96"/>
+</instance>
 </instances>
 <busses>
@@
 <junction x="284.48" y="58.42"/>
 <pinref part="L2" gate="G$1" pin="1"/>
+<pinref part="C71" gate="G$1" pin="1"/>
+<wire x1="238.76" y1="68.58" x2="238.76" y2="71.12" width="0.1524" layer="91"/>
+<junction x="238.76" y="71.12"/>
 </segment>
 </net>
@@
 <wire x1="284.48" y1="149.86" x2="238.76" y2="149.86" width="0.1524" layer="91"/>
 <wire x1="238.76" y1="149.86" x2="238.76" y2="129.54" width="0.1524" layer="91"/>
+<pinref part="C68" gate="G$1" pin="1"/>
+<wire x1="238.76" y1="127" x2="238.76" y2="129.54" width="0.1524" layer="91"/>
+<junction x="238.76" y="129.54"/>
 </segment>
 </net>
@@
 <wire x1="254" y1="116.84" x2="238.76" y2="116.84" width="0.1524" layer="91"/>
 <junction x="254" y="116.84"/>
+<pinref part="C68" gate="G$1" pin="2"/>
+<wire x1="238.76" y1="116.84" x2="238.76" y2="121.92" width="0.1524" layer="91"/>
+<junction x="238.76" y="116.84"/>
 </segment>
 </net>
@@
 <wire x1="254" y1="58.42" x2="238.76" y2="58.42" width="0.1524" layer="91"/>
 <junction x="254" y="58.42"/>
+<pinref part="C71" gate="G$1" pin="2"/>
+<wire x1="238.76" y1="58.42" x2="238.76" y2="63.5" width="0.1524" layer="91"/>
+<junction x="238.76" y="58.42"/>
 </segment>
 </net>

Commit message: 微修正
Parts:
- removed TP15, TP16: +12V, my_connector:TESTPIN
- removed TP17, TP20: SW_SP, my_connector:TESTPIN
- removed TP18, TP19: SW_HP, my_connector:TESTPIN
- TP31: value GND_L -> GND
Connections:
- net +12VD: no longer TP15.1, TP16.1
- net HP_L: now also SW2.COM2; no longer SW2.COM1
- net HP_R: now also SW2.COM1; no longer SW2.COM2
- net N$33: now also SW1.A1, SW2.A1; no longer SW1.A2, SW2.A2
- net N$34: now also SW1.A2, SW2.A2; no longer SW1.A1, SW2.A1
- net SPK_L: now also SW1.COM2; no longer SW1.COM1
- net SPK_R: now also SW1.COM1; no longer SW1.COM2
- net SW_HP: no longer TP18.1, TP19.1
- net SW_SP: no longer TP17.1, TP20.1
Other:
- moved on the sheet: D8, Q6, R59, R60, SW1, SW2

Commit message: Add 位相補償
Parts:
- added C74, C75: CMP, my_rcl:C-1608
Connections:
- net N$21: now also C75.1
- net N$26: now also C75.2
- net N$44: now also C74.1
- net N$53: now also C74.2
Other:
- moved on the sheet: C69, C70, R39, R40, R43, R44

Commit message: 微修正
Parts:
- removed DECO1: ROBOTECH_WHEEL, my_connector:ROBOTECH_WHEEL
- added R33, R34, R45, R46: 10, my_rcl:R-1608
- IC19, IC23, IC8: value (none) -> ADA4075
- R17: value 10k0.1% -> 10k
Connections:
- new net DAC_NRST: IC13.DP28, IC7.!RST
- new net N$51: Q10.E, R33.2
- new net N$56: D5.K, Q3.B, R34.2, R51.1
- new net N$57: Q7.E, R45.2
- new net N$58: Q8.E, R46.1
- net N$16: now also R45.1; no longer Q7.E
- net N$29: now also R34.1; no longer D5.K, Q3.B, R51.1
- net N$49: now also R46.2; no longer Q8.E
- net N$54: now also R33.1; no longer Q10.E
Other:
- moved on the sheet: C63, C67, C68, C69, C70, C71, C74, C75, D3, D4, D5, D6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

Commit message: fix PCM1795
Parts:
- C15: value 10u -> 2.2u
- C18: value 0.1u -> 1000p
- C4, C5: value 22p -> 10p
- C40, C42: device my_rcl:C-1608 -> my_rcl:C-2012
Connections:
- net DAC_MCLK/2: now also IC3.IN1; no longer IC3.IN2
- net GND: now also IC3.IN2; no longer IC3.IN1

Commit message: 微修正
Parts:
- added R47, R48: 10, my_rcl:R-2012
Connections:
- net AMP_LOUT: now also R47.1
- net AMP_ROUT: now also R48.1
- net N$33: now also R48.2
- net N$34: now also R47.2

Commit message: AK4495に変える
Parts:
- removed C34: 0.1u, my_rcl:C-1608
- removed IC8: ADA4075, my_ic:OPA-2-SOP
- removed R17: 10k, my_rcl:R-1608
- removed R18, R19, R20, R21: 1k, my_rcl:R-1608
- removed R22, R23, R24, R25: 10, my_rcl:R-1608J
- added FB7: FB, my_rcl:FB
- C40: value 0.1u -> 100u; device my_rcl:C-2012 -> my_rcl:CPOLE2.5-6.5
- C42: value 0.1u -> 10u
- C45, C53, C57: value 0.1u -> 100u; device my_rcl:C-1608 -> my_rcl:CPOLE2.5-6.5
- C46: value 0.1u -> 220u; device my_rcl:C-1608 -> my_rcl:CPOLE2.5-6.5
- C47, C48, C54, C55: value 100u -> 0.1u; device my_rcl:CPOLE2.5-6.5 -> my_rcl:C-1608
- C49, C50, C52: value 3300p -> 0.1u
- C51: value 3300p -> 100u; device my_rcl:C-1608 -> my_rcl:CPOLE2.5-6.5
- C58: value 100u -> 220u
- IC19: value ADA4075 -> AK4495EQ; device my_ic:OPA-2-SOP -> my_ic:AK4495EQ
- IC7: value PCM1795 -> +5V; device my_ic:PCM1795 -> my_ic:78X-LED
Connections:
- removed net IOUTL+: IC7.IOUTL+, R25.1
- removed net IOUTL-: IC7.IOUTL-, R24.1
- removed net IOUTR+: IC7.IOUTR+, R23.1
- removed net IOUTR-: IC7.IOUTR-, R22.1
- removed net N$14: C58.2, IC7.VCOMR
- removed net N$27: IC7.IREF, R17.2
- removed net N$37: C47.2, IC7.VCOML
- removed net N$41: C49.1, IC8G$1.-IN, R18.1, R22.2
- removed net N$42: C50.1, IC8G$2.-IN, R19.1, R23.2
- removed net N$43: C51.1, IC19G$1.-IN, R20.1, R24.2
- removed net N$55: C52.1, IC19G$2.-IN, R21.1, R25.2
- new net DAC_AVDD: IC19.DEM0, IC19.I2C
- new net DAC_DVDD: C42.1, C48.1, FB7.2, IC19.DVDD
- new net DAC_PDN: IC19.PDN
- new net DAC_VREF: C30.2, C46.1, C50.2, C58.1, IC19.VREFHL1, IC19.VREFHL2, IC19.VREFHR1, IC19.VREFHR2, IC7.OUT
- new net VCOM_L: C45.1, C49.1, IC19.VCOML
- new net VCOM_R: C55.1, C57.1, IC19.VCOMR
- net +12V: now also IC7.IN
- net DAC_DATA: now also IC19.SDATA; no longer IC7.DATA
- net DAC_LN: now also IC19.OUTLN; no longer C52.2, IC19G$2.OUT, R21.2
- net DAC_LP: now also IC19.OUTLP; no longer C51.2, IC19G$1.OUT, R20.2
- net DAC_LRCLK: now also IC19.LRCK; no longer IC7.LRCK
- net DAC_MCLK: now also IC19.MCLK; no longer IC7.SCK
- net DAC_NRST: no longer IC7.!RST
- net DAC_RN: now also IC19.OUTRN; no longer C50.2, IC8G$2.OUT, R19.2
- net DAC_RP: now also IC19.OUTRP; no longer C49.2, IC8G$1.OUT, R18.2
- net DAC_SCK: now also IC19.BCK; no longer IC7.BCK
- net DAC_VCC: now also C51.1, C52.1, C53.1, C54.1, IC19.VDDL1, IC19.VDDL2, IC19.VDDR1, IC19.VDDR2; no longer C40.1, C42.1, C45.1, C47.1, C48.1, C55.1, C58.1, IC7.VCC1, IC7.VCC2L, IC7.VCC2R
- net DAC_VDD: now also C40.1, C47.1, FB7.1, IC19.AVDD; no longer C53.1, C54.1, IC7.MSEL, IC7.VDD
- net GND: now also C30.1, C46.2, C47.2, C49.2, C50.1, C51.2, C52.2, C57.2, C58.2, IC19.ACKS/CAD1, IC19.AVSS, IC19.DEM1, IC19.DIF2/CAD0, IC19.DVSS, IC19.NC, IC19.PSN, IC19.SMUTE/CSN, IC19.SSLOW, IC19.VREFLL1, IC19.VREFLL2, IC19.VREFLR1, IC19.VREFLR2, IC19.VSSL1, IC19.VSSL2, IC19.VSSR1, IC19.VSSR2, IC7.GND; no longer C30.2, C34.2, C46.1, C57.1, IC19G$1.+IN, IC19G$2.+IN, IC7.!MS, IC7.AGND1, IC7.AGND2, IC7.AGND3L, IC7.AGND3R, IC7.DGND, IC7.MDI, IC8G$1.+IN, IC8G$2.+IN, R17.1
- net I2C_SCL: now also IC19.SD/SCL; no longer IC7.MC
- net I2C_SDA: now also IC19.SLOW/SDA; no longer IC7.MDO
- net OPA_+: no longer C30.1, C34.1, IC19G$3.V+, IC8G$3.V+
- net OPA_-: no longer C46.2, C57.2, IC19G$3.V-, IC8G$3.V-
Other:
- moved on the sheet: C30, C42, C49, C50, C52, C58, IC17, IC23G$3

Commit message: できた
Connections:
- removed net DAC_AVDD: IC19.DEM0, IC19.I2C
- removed net DAC_NRST: IC13.DP28
- removed net N$47: IC4.OUT1, R26.1
- new net N$14: IC5.OUT1, R30.1
- net DAC_DVDD: now also IC19.DEM0, IC19.I2C
- net DAC_LRCLK: now also R26.2; no longer R30.2
- net DAC_LRCLK_IN: now also IC4.OUT1, R26.1; no longer IC5.OUT1, R30.1
- net DAC_PDN: now also IC13.DP28
- net DAC_SCK: now also R30.2; no longer R26.2
- net D_LRCLK: now also IC4.IN1; no longer IC5.IN1
- net D_SCK: now also IC5.IN1; no longer IC4.IN1
